File: bottom-board/audio-codec.sch (KiCad schematic (older format))
At the start: 45 parts, among them U13 AP2120N-3.3, U3 CODECODER-WM8731SEDS_V(SSOP28)

Commit message: add fabrication files bottom board
Parts:
- C13, C14, C26: MPN (none) -> UWX1H010MCL2GB
- C20, C21: footprint Capacitor_SMD:CP_Elec_10x7.9 -> Capacitor_SMD:CP_Elec_6.3x5.4; MPN (none) -> ECE-V0JA221WP
- C27: footprint Capacitor_SMD:C_0402_1005Metric -> Capacitor_SMD:C_0603_1608Metric; MPN (none) -> CC0603KRX7R9BB221
- C28: renamed from CA1; MPN (none) -> CC0603KRX7R9BB221
- C29: renamed from CA2; MPN (none) -> CC0603KRX7R9BB221
- R11, R8: value 100 -> 100R; MPN (none) -> RMCF0603JT100R
- R13, R14, R15, R17, R23: MPN (none) -> RC0603JR-0747KL
- R16: MPN (none) -> CR0603-JW-471ELF
- R19, R20, R21, R22: MPN RMCF0603JT22R0 -> RMCF0603JT5K60
- U13: MPN (none) -> AP2120N-3.3TRG1
- U3: Field4 Unavailable -> (none); Field5 None -> (none); Field6 SSOP-28 Cirrus Logic -> (none); Field7 WM8731SEDS/V -> (none); Field8 Audio Codec 2ADC /2 DAC 24-Bit 28-Pin SSOP -> (none); MPN (none) -> WM8731SEDS/V
Changed lines of the file:
@@
 F 2 "Package_TO_SOT_SMD:SOT-23" H 2000 1600 50  0001 C CNN
 F 3 "https://www.diodes.com/assets/Datasheets/AP2120.pdf" H 2100 1150 50  0001 C CNN
+F 4 "AP2120N-3.3TRG1" H 2000 1400 50  0001 C CNN "MPN"
 	1    2000 1400
 	1    0    0    -1
@@
 F 2 "Resistor_SMD:R_0603_1608Metric" H 7750 3600 60  0001 C CNN
 F 3 "" H 7750 3600 60  0000 C CNN
-F 4 "RMCF0603JT22R0" H 3450 1250 50  0001 C CNN "MPN"
+F 4 "RMCF0603JT5K60" H 3450 1250 50  0001 C CNN "MPN"
 	1    7750 3600
 	0    1    1    0
@@
 F 2 "Resistor_SMD:R_0603_1608Metric" H 7750 3700 60  0001 C CNN
 F 3 "" H 7750 3700 60  0000 C CNN
-F 4 "RMCF0603JT22R0" H 3450 1350 50  0001 C CNN "MPN"
+F 4 "RMCF0603JT5K60" H 3450 1350 50  0001 C CNN "MPN"
 	1    7750 3700
 	0    1    1    0
@@
 F 2 "Resistor_SMD:R_0603_1608Metric" H 7500 3850 60  0001 C CNN
 F 3 "" H 7500 3850 60  0000 C CNN
-F 4 "RMCF0603JT22R0" H 3200 1500 50  0001 C CNN "MPN"
+F 4 "RMCF0603JT5K60" H 3200 1500 50  0001 C CNN "MPN"
 	1    7500 3850
 	-1   0    0    1
@@
 F 2 "Resistor_SMD:R_0603_1608Metric" H 7150 3850 60  0001 C CNN
 F 3 "" H 7150 3850 60  0000 C CNN
-F 4 "RMCF0603JT22R0" H 2850 1500 50  0001 C CNN "MPN"
+F 4 "RMCF0603JT5K60" H 2850 1500 50  0001 C CNN "MPN"
 	1    7150 3850
 	-1   0    0    1
 $EndComp
 $Comp
-L bottom-board-rescue:C_Small CA2
+L bottom-board-rescue:C_Small C29
 U 1 1 5DEE68B9
 P 7350 3850
-F 0 "CA2" V 7300 3650 50  0000 L CNN
+F 0 "C29" V 7300 3650 50  0000 L CNN
 F 1 "220pF" V 7400 3600 50  0000 L CNN
 F 2 "Capacitor_SMD:C_0603_1608Metric" H 7350 3850 60  0001 C CNN
 F 3 "" H 7350 3850 60  0000 C CNN
-F 4 "" H 2250 -1500 50  0001 C CNN "MPN"
+F 4 "CC0603KRX7R9BB221" H 2250 -1500 50  0001 C CNN "MPN"
 	1    7350 3850
 	1    0    0    -1
 $EndComp
 $Comp
-L bottom-board-rescue:C_Small CA1
+L bottom-board-rescue:C_Small C28
 U 1 1 5DEE741E
 P 7000 3850
-F 0 "CA1" V 6950 3650 50  0000 L CNN
+F 0 "C28" V 6950 3650 50  0000 L CNN
 F 1 "220pF" V 7075 3625 50  0000 L CNN
 F 2 "Capacitor_SMD:C_0603_1608Metric" H 7000 3850 60  0001 C CNN
 F 3 "" H 7000 3850 60  0000 C CNN
-F 4 "" H 1900 -1500 50  0001 C CNN "MPN"
+F 4 "CC0603KRX7R9BB221" H 1900 -1500 50  0001 C CNN "MPN"
 	1    7000 3850
 	1    0    0    -1
@@
 F 2 "Capacitor_SMD:CP_Elec_3x5.4" H 5250 3900 60  0001 C CNN
 F 3 "" H 5250 3900 60  0000 C CNN
-F 4 "" H 150 2400 50  0001 C CNN "MPN"
+F 4 "UWX1H010MCL2GB" H 150 2400 50  0001 C CNN "MPN"
 	1    5250 3900
 	0    1    1    0
@@
 F 2 "Capacitor_SMD:CP_Elec_3x5.4" H 5250 4000 60  0001 C CNN
 F 3 "" H 5250 4000 60  0000 C CNN
-F 4 "" H 150 2500 50  0001 C CNN "MPN"
+F 4 "UWX1H010MCL2GB" H 150 2500 50  0001 C CNN "MPN"
 	1    5250 4000
 	0    1    1    0
@@
 P 4850 4000
 F 0 "R11" V 4750 3950 50  0000 R CNN
-F 1 "100" V 4750 4000 50  0000 L CNN
+F 1 "100R" V 4750 4000 50  0000 L CNN
 F 2 "Resistor_SMD:R_0603_1608Metric" H 4850 4000 60  0001 C CNN
 F 3 "" H 4850 4000 60  0000 C CNN
-F 4 "" H -700 2600 50  0001 C CNN "MPN"
+F 4 "RMCF0603JT100R" H -700 2600 50  0001 C CNN "MPN"
 	1    4850 4000
 	0    -1   -1   0
@@
 P 4850 3900
 F 0 "R8" V 4900 3850 50  0000 R CNN
-F 1 "100" V 4900 3900 50  0000 L CNN
+F 1 "100R" V 4900 3900 50  0000 L CNN
 F 2 "Resistor_SMD:R_0603_1608Metric" H 4850 3900 60  0001 C CNN
 F 3 "" H 4850 3900 60  0000 C CNN
-F 4 "" H -700 2500 50  0001 C CNN "MPN"
+F 4 "RMCF0603JT100R" H -700 2500 50  0001 C CNN "MPN"
 	1    4850 3900
 	0    -1   -1   0
@@
 F 2 "Resistor_SMD:R_0603_1608Metric" H 5100 4250 60  0001 C CNN
 F 3 "" H 5100 4250 60  0000 C CNN
-F 4 "" H -450 2850 50  0001 C CNN "MPN"
+F 4 "RC0603JR-0747KL" H -450 2850 50  0001 C CNN "MPN"
 	1    5100 4250
 	-1   0    0    1
@@
 F 2 "Resistor_SMD:R_0603_1608Metric" H 5000 4250 60  0001 C CNN
 F 3 "" H 5000 4250 60  0000 C CNN
-F 4 "" H -550 2850 50  0001 C CNN "MPN"
+F 4 "RC0603JR-0747KL" H -550 2850 50  0001 C CNN "MPN"
 	1    5000 4250
 	-1   0    0    1
@@
 F 0 "C20" V 4625 3400 50  0000 L CNN
 F 1 "220uF" V 4625 3650 50  0000 L CNN
-F 2 "Capacitor_SMD:CP_Elec_10x7.9" H 4575 3600 60  0001 C CNN
+F 2 "Capacitor_SMD:CP_Elec_6.3x5.4" H 4575 3600 60  0001 C CNN
 F 3 "" H 4575 3600 60  0000 C CNN
-F 4 "" H -525 2100 50  0001 C CNN "MPN"
+F 4 "ECE-V0JA221WP" H -525 2100 50  0001 C CNN "MPN"
 	1    4575 3600
 	0    1    1    0
@@
 F 0 "C21" V 4625 3500 50  0000 L CNN
 F 1 "220uF" V 4625 3750 50  0000 L CNN
-F 2 "Capacitor_SMD:CP_Elec_10x7.9" H 4575 3700 60  0001 C CNN
+F 2 "Capacitor_SMD:CP_Elec_6.3x5.4" H 4575 3700 60  0001 C CNN
 F 3 "" H 4575 3700 60  0000 C CNN
-F 4 "" H -525 2200 50  0001 C CNN "MPN"
+F 4 "ECE-V0JA221WP" H -525 2200 50  0001 C CNN "MPN"
 	1    4575 3700
 	0    1    1    0
@@
 F 2 "Resistor_SMD:R_0603_1608Metric" H 3875 3900 60  0001 C CNN
 F 3 "" H 3875 3900 60  0000 C CNN
-F 4 "" H -1675 2500 50  0001 C CNN "MPN"
+F 4 "RC0603JR-0747KL" H -1675 2500 50  0001 C CNN "MPN"
 	1    3875 3900
 	-1   0    0    1
@@
 F 2 "Resistor_SMD:R_0603_1608Metric" H 3775 3900 60  0001 C CNN
 F 3 "" H 3775 3900 60  0000 C CNN
-F 4 "" H -1775 2500 50  0001 C CNN "MPN"
+F 4 "RC0603JR-0747KL" H -1775 2500 50  0001 C CNN "MPN"
 	1    3775 3900
 	-1   0    0    1
@@
 F 2 "Capacitor_SMD:CP_Elec_3x5.4" H 9250 3800 60  0001 C CNN
 F 3 "" H 9250 3800 60  0000 C CNN
-F 4 "" H 4150 2300 50  0001 C CNN "MPN"
+F 4 "UWX1H010MCL2GB" H 4150 2300 50  0001 C CNN "MPN"
 	1    9250 3800
 	0    -1   -1   0
@@
 F 2 "Resistor_SMD:R_0603_1608Metric" H 9450 3975 60  0001 C CNN
 F 3 "" H 9450 3975 60  0000 C CNN
+F 4 "RC0603JR-0747KL" V 9450 3975 50  0001 C CNN "MPN"
 	1    9450 3975
 	-1   0    0    1
@@
 F 0 "C27" V 9725 3850 50  0000 L CNN
 F 1 "220pF" V 9800 3900 50  0000 L CNN
-F 2 "Capacitor_SMD:C_0402_1005Metric" H 9650 4000 60  0001 C CNN
+F 2 "Capacitor_SMD:C_0603_1608Metric" H 9650 4000 60  0001 C CNN
 F 3 "" H 9650 4000 60  0000 C CNN
+F 4 "CC0603KRX7R9BB221" V 9650 4000 50  0001 C CNN "MPN"
 	1    9650 4000
 	1    0    0    -1
@@
 F 2 "Resistor_SMD:R_0603_1608Metric" H 8800 3800 60  0001 C CNN
 F 3 "" H 8800 3800 60  0000 C CNN
+F 4 "CR0603-JW-471ELF" V 8800 3800 50  0001 C CNN "MPN"
 	1    8800 3800
 	0    1    1    0
@@
 F 2 "SSOP28-0.65-10.2X5.2MM" H 6150 3450 50  0001 L BNN
 F 3 "" H 6150 3450 50  0001 L BNN
-F 4 "Unavailable" H 6150 3450 50  0001 L BNN "Field4"
-F 5 "None" H 6150 3450 50  0001 L BNN "Field5"
-F 6 "SSOP-28 Cirrus Logic" H 6150 3450 50  0001 L BNN "Field6"
-F 7 "WM8731SEDS/V" H 6150 3450 50  0001 L BNN "Field7"
-F 8 "Audio Codec 2ADC /2 DAC 24-Bit 28-Pin SSOP" H 6150 3450 50  0001 L BNN "Field8"
+F 4 "WM8731SEDS/V" H 6150 3450 50  0001 C CNN "MPN"
 	1    6150 3450
 	1    0    0    -1
