File: bottom-board/audio-inputs.sch (KiCad schematic (older format))
At the start: 11 parts, among them Q1 J110, Q2 J110, U5 TS5A3159ADBVR

Commit message: add fabrication files bottom board
Parts:
- Q1, Q2: MPN (none) -> MMBFJ110
- R24, R25: MPN RMCF0603JT22R0 -> RMCF0603JT5K60
- U5: MPN (none) -> TS5A3159ADBVR
- renumbered CA3 to C33, CA4 to C34, CA5 to C35, CA6 to C36, RA4 to R31, RA2 to R32
Changed lines of the file:
@@
 CODEC_ADC_B
 $Comp
-L bottom-board-rescue:R_Small RA4
+L bottom-board-rescue:R_Small R31
 U 1 1 5D47C4D2
 P 5050 2925
-F 0 "RA4" H 5100 2975 50  0000 L CNN
+F 0 "R31" H 5100 2975 50  0000 L CNN
 F 1 "1M" H 5100 2875 50  0000 L CNN
 F 2 "Resistor_SMD:R_0603_1608Metric" H 5050 2925 60  0001 C CNN
@@
 	5050 2825 5050 2675
 $Comp
-L bottom-board-rescue:CP_Small CA3
+L bottom-board-rescue:CP_Small C33
 U 1 1 5D4C57FE
 P 4750 2675
-F 0 "CA3" H 4850 2675 50  0000 L CNN
+F 0 "C33" H 4850 2675 50  0000 L CNN
 F 1 "10uF" H 4800 2575 50  0000 L CNN
 F 2 "Capacitor_SMD:CP_Elec_5x5.3" H 4750 2675 60  0001 C CNN
@@
 Connection ~ 5050 2675
 $Comp
-L bottom-board-rescue:CP_Small CA5
+L bottom-board-rescue:CP_Small C35
 U 1 1 5D530CBE
 P 5900 2950
-F 0 "CA5" H 6000 2950 50  0000 L CNN
+F 0 "C35" H 6000 2950 50  0000 L CNN
 F 1 "10uF" H 5950 2850 50  0000 L CNN
 F 2 "Capacitor_SMD:CP_Elec_5x5.3" H 5900 2950 60  0001 C CNN
@@
 F 2 "Package_TO_SOT_SMD:SOT-23" H 5650 2775 50  0001 C CNN
 F 3 "https://www.nxp.com/docs/en/data-sheet/PMBFJ108_109_110.pdf" H 5450 2675 50  0001 C CNN
+F 4 "MMBFJ110" H 5450 2675 50  0001 C CNN "MPN"
 	1    5450 2675
 	1    0    0    -1
@@
 F 2 "Resistor_SMD:R_0603_1608Metric" H 5550 3125 60  0001 C CNN
 F 3 "" H 5550 3125 60  0000 C CNN
-F 4 "RMCF0603JT22R0" H 1250 775 50  0001 C CNN "MPN"
+F 4 "RMCF0603JT5K60" H 1250 775 50  0001 C CNN "MPN"
 	1    5550 3125
 	1    0    0    -1
@@
 	5550 2950 5550 2875
 $Comp
-L bottom-board-rescue:R_Small RA2
+L bottom-board-rescue:R_Small R32
 U 1 1 5DDE85CA
 P 5075 4475
-F 0 "RA2" H 5125 4525 50  0000 L CNN
+F 0 "R32" H 5125 4525 50  0000 L CNN
 F 1 "1M" H 5125 4425 50  0000 L CNN
 F 2 "Resistor_SMD:R_0603_1608Metric" H 5075 4475 60  0001 C CNN
@@
 	5075 4375 5075 4225
 $Comp
-L bottom-board-rescue:CP_Small CA4
+L bottom-board-rescue:CP_Small C34
 U 1 1 5DDE85D2
 P 4775 4225
-F 0 "CA4" H 4875 4225 50  0000 L CNN
+F 0 "C34" H 4875 4225 50  0000 L CNN
 F 1 "10uF" H 4825 4125 50  0000 L CNN
 F 2 "Capacitor_SMD:CP_Elec_5x5.3" H 4775 4225 60  0001 C CNN
@@
 Connection ~ 5075 4225
 $Comp
-L bottom-board-rescue:CP_Small CA6
+L bottom-board-rescue:CP_Small C36
 U 1 1 5DDE85DB
 P 5925 4500
-F 0 "CA6" H 6025 4500 50  0000 L CNN
+F 0 "C36" H 6025 4500 50  0000 L CNN
 F 1 "10uF" H 5975 4400 50  0000 L CNN
 F 2 "Capacitor_SMD:CP_Elec_5x5.3" H 5925 4500 60  0001 C CNN
@@
 F 2 "Package_TO_SOT_SMD:SOT-23" H 5675 4325 50  0001 C CNN
 F 3 "https://www.nxp.com/docs/en/data-sheet/PMBFJ108_109_110.pdf" H 5475 4225 50  0001 C CNN
+F 4 "MMBFJ110" H 5475 4225 50  0001 C CNN "MPN"
 	1    5475 4225
 	1    0    0    -1
@@
 F 2 "Resistor_SMD:R_0603_1608Metric" H 5575 4675 60  0001 C CNN
 F 3 "" H 5575 4675 60  0000 C CNN
-F 4 "RMCF0603JT22R0" H 1275 2325 50  0001 C CNN "MPN"
+F 4 "RMCF0603JT5K60" H 1275 2325 50  0001 C CNN "MPN"
 	1    5575 4675
 	1    0    0    -1
@@
 F 2 "Package_TO_SOT_SMD:SOT-23-6" H 4050 2375 50  0001 C CNN
 F 3 "http://www.ti.com/lit/ds/symlink/ts5a3159a.pdf" H 4050 2675 50  0001 C CNN
+F 4 "TS5A3159ADBVR" H 4050 2675 50  0001 C CNN "MPN"
 	1    4050 2675
 	1    0    0    -1
