File: bottom-board/bottom-board.kicad_pcb (KiCad board)
At the start: 2 copper layers, 184 x 94 mm, 155 parts, among them J1 AS0A823-H4SB-7H, P1 USB_B, P10 JACK_TRS_6PINS, P11 JACK_TRS_6PINS, P12 JACK_TRS_6PINS, P13 JACK_TRS_6PINS, P14 RJ45, P2 USB_A, P3 AudioJack3, P5 BARREL_JACK, P6 AudioJack3, P7 AudioJack3, P8 HMI_DATA, P9 SERIAL_DEBUG, Q1 J110, Q12 2N7002, Q13 2N7002, Q2 J110, U1 TS2596, U10 RT9742MNGJ5, U11 6N137S, U12 ISL83491, U13 AP2120N-3.3, U2 LD1117S50TR_SOT223, U3 CODECODER-WM8731SEDS_V(SSOP28), U4 AT24CS08-STUM, U5 TS5A3159ADBVR

Commit message: add fabrication files bottom board
Parts:
- removed G***: LOGO, Uno:mod-logo
- removed J1: AS0A823-H4SB-7H, Uno:FOXCONN_AS0A823-H4SB-7H
- removed Revocery: TestPoint, TestPoint:TestPoint_Pad_D3.0mm
- added H8: HOLE, MountingHole:MountingHole_3mm, F.Cu at (104.2, 72.3)
- added H9: HOLE, MountingHole:MountingHole_3mm, F.Cu at (70.3, 106.3)
- added P4: AS0A823-H4SB-7H, Uno:TE_2309407-1, F.Cu at (104.4, 117.7)
- added TP2: TestPoint, TestPoint:TestPoint_Pad_D1.5mm, B.Cu at (107.0, 109.4)
- C20, C21: footprint Capacitor_SMD:CP_Elec_10x7.9 -> Capacitor_SMD:CP_Elec_6.3x5.4
- C27: footprint Capacitor_SMD:C_0402_1005Metric -> Capacitor_SMD:C_0603_1608Metric
- L2: value INDUCTOR -> 47UH 2A 135 MOHM
- R11, R8: value 100 -> 100R
- R30: renamed from RA1; value 10 -> 10R
- R42: value 5k6 -> 5K6
- R47: footprint Resistor_SMD:R_0805_2012Metric -> Resistor_SMD:R_0603_1608Metric
- TP1: footprint TestPoint:TestPoint_Pad_D3.0mm -> TestPoint:TestPoint_Pad_D1.5mm
- moved C34 4.20 mm to (219.2, 69.9)
- moved H7 2.77 mm to (133.2, 72.6)
- moved H6 2.37 mm to (68.6, 72.7)
- moved R15 2.24 mm to (192.0, 100.3)
- moved R14 2.24 mm to (192.0, 105.2)
- moved C33 2.07 mm to (231.5, 70.6)
- moved Q1 1.86 mm to (234.6, 75.6)
- moved P11 1.31 mm to (203.3, 58.7)
- moved P13 1.28 mm to (82.5, 58.7)
- moved P10 1.22 mm to (223.6, 58.6)
- moved P12 1.13 mm to (102.7, 58.5)
- moved R32 1.08 mm to (226.8, 71.6), turned to 90 degrees
- moved R24 0.62 mm to (237.3, 75.5), turned to 90 degrees
- moved R47 0.07 mm to (192.2, 56.4), turned to 0 degrees
- renumbered CA1 to C28, CA2 to C29, CA3 to C33, CA4 to C34, CA5 to C35, CA6 to C36, RA4 to R31, RA2 to R32
Connections:
- R47 pad 1: Net-(D15-Pad1) -> Net-(P6-PadT)
- R47 pad 2: Net-(P6-PadT) -> Net-(D15-Pad1)
Routing:
- net GNDA: track 356.7 -> 431.5 mm, vias 76 -> 77
- net RIGHT_AUDIO_INPUT: track 27.2 -> 22.8 mm
- net OUT2_DETECT: track 114.4 -> 110.1 mm
- net Net-(C34-Pad1): track 6.93 -> 11.2 mm
- net +5VA: track 125.5 -> 127.9 mm
- net IN1_DETECT: track 209.0 -> 207.2 mm
- net MIC_SELECT: track 175.1 -> 176.5 mm
- net HEADPHONE_RIGHT: track 147.2 -> 148.5 mm
- net Net-(C35-Pad2): track 5.94 -> 6.91 mm
- net Net-(R30-Pad2): track 1.10 -> 2.06 mm
- net CODEC_DAC_A: track 152.1 -> 151.2 mm
- net CHAIN_UART_RX: track 130.5 -> 131.4 mm
- net Net-(C33-Pad2): track 9.65 -> 10.4 mm
- net +5V: track 259.9 -> 260.6 mm
- net CODEC_DAC_B: track 156.2 -> 155.5 mm
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Other:
- board text added: "GND RX TX"
- board text added: "Recovery"
