File: bottom-board/connectors.sch (KiCad schematic (older format))
At the start: 18 parts, among them P10 JACK_TRS_6PINS, P11 JACK_TRS_6PINS, P12 JACK_TRS_6PINS, P13 JACK_TRS_6PINS, P14 RJ45, P3 AudioJack3, P5 BARREL_JACK, P8 HMI_DATA, P9 SERIAL_DEBUG

Commit message: add fabrication files bottom board
Parts:
- P10, P11, P12, P13: MPN NMJ6HCD2 -> NYS215
- P14: MPN (none) -> 54602-908LF
- P3: MPN (none) -> SJ-3523-SMT-TR
- P9: MPN (none) -> DO NOT PLACE
- R26, R27, R28, R29: MPN (none) -> CR0603-JW-104ELF
Changed lines of the file:
@@
 F 2 "Connector_PinHeader_2.54mm:PinHeader_1x03_P2.54mm_Vertical" H 9750 2650 60  0001 C CNN
 F 3 "" H 9750 2650 60  0000 C CNN
+F 4 "DO NOT PLACE" H 9750 2650 50  0001 C CNN "MPN"
 	1    9750 2650
 	1    0    0    -1
@@
 F 2 "Connector_Audio:Jack_3.5mm_Neutrik_NMJ6HCD2_Horizontal" H 2050 5350 60  0001 C CNN
 F 3 "" H 2050 5350 60  0000 C CNN
-F 4 "NMJ6HCD2" H 0   -200 50  0001 C CNN "MPN"
+F 4 "NYS215" H 0   -200 50  0001 C CNN "MPN"
 	1    1900 5500
 	1    0    0    -1
@@
 F 2 "Connector_Audio:Jack_3.5mm_Neutrik_NMJ6HCD2_Horizontal" H 2050 4500 60  0001 C CNN
 F 3 "" H 2050 4500 60  0000 C CNN
-F 4 "NMJ6HCD2" H 0   -200 50  0001 C CNN "MPN"
+F 4 "NYS215" H 0   -200 50  0001 C CNN "MPN"
 	1    1900 4650
 	1    0    0    -1
@@
 F 2 "Connector_Audio:Jack_3.5mm_Neutrik_NMJ6HCD2_Horizontal" H 5450 4500 60  0001 C CNN
 F 3 "" H 5450 4500 60  0000 C CNN
-F 4 "NMJ6HCD2" H 0   -200 50  0001 C CNN "MPN"
+F 4 "NYS215" H 0   -200 50  0001 C CNN "MPN"
 	1    5300 4650
 	-1   0    0    -1
@@
 F 2 "Connector_Audio:Jack_3.5mm_Neutrik_NMJ6HCD2_Horizontal" H 5450 5350 60  0001 C CNN
 F 3 "" H 5450 5350 60  0000 C CNN
-F 4 "NMJ6HCD2" H 0   -200 50  0001 C CNN "MPN"
+F 4 "NYS215" H 0   -200 50  0001 C CNN "MPN"
 	1    5300 5500
 	-1   0    0    -1
@@
 F 2 "Resistor_SMD:R_0603_1608Metric" H 2400 4350 60  0001 C CNN
 F 3 "" H 2400 4350 60  0000 C CNN
+F 4 "CR0603-JW-104ELF" H 2400 4350 50  0001 C CNN "MPN"
 	1    2400 4350
 	1    0    0    -1
@@
 F 2 "Resistor_SMD:R_0603_1608Metric" H 2400 5200 60  0001 C CNN
 F 3 "" H 2400 5200 60  0000 C CNN
+F 4 "CR0603-JW-104ELF" H 2400 5200 50  0001 C CNN "MPN"
 	1    2400 5200
 	1    0    0    -1
@@
 F 2 "Resistor_SMD:R_0603_1608Metric" H 4650 4375 60  0001 C CNN
 F 3 "" H 4650 4375 60  0000 C CNN
+F 4 "CR0603-JW-104ELF" H 4650 4375 50  0001 C CNN "MPN"
 	1    4650 4375
 	-1   0    0    1
@@
 F 2 "Resistor_SMD:R_0603_1608Metric" H 4650 5225 60  0001 C CNN
 F 3 "" H 4650 5225 60  0000 C CNN
+F 4 "CR0603-JW-104ELF" H 4650 5225 50  0001 C CNN "MPN"
 	1    4650 5225
 	-1   0    0    1
@@
 F 2 "Connector_Audio:Jack_3.5mm_CUI_SJ-3523-SMT_Horizontal" H 1625 2825 50  0001 C CNN
 F 3 "~" H 1625 2825 50  0001 C CNN
+F 4 "SJ-3523-SMT-TR" V 1625 2825 50  0001 C CNN "MPN"
 	1    1625 2825
 	1    0    0    -1
@@
 F 2 "digikey-footprints:Ethernet_Jack_54602-908LF" V 8450 4675 50  0001 C CNN
 F 3 "~" V 8450 4675 50  0001 C CNN
+F 4 "54602-908LF" H 8450 4650 50  0001 C CNN "MPN"
 	1    8450 4650
 	-1   0    0    1
