File: bottom-board/control-chain.sch (KiCad schematic (older format))
At the start: 11 parts, among them U12 ISL83491

Commit message: add fabrication files bottom board
Parts:
- R63: MPN ERJ-P06J101V -> RMCF0603JT100R
Changed lines of the file:
@@
 F 2 "Resistor_SMD:R_0603_1608Metric" H 6650 3300 60  0001 C CNN
 F 3 "" H 6650 3300 60  0000 C CNN
-F 4 "ERJ-P06J101V" H 100 1000 50  0001 C CNN "MPN"
+F 4 "RMCF0603JT100R" H 100 1000 50  0001 C CNN "MPN"
 	1    6650 3300
 	1    0    0    -1
