File: bottom-board/mechanics.sch (KiCad schematic (older format))
At the start: 10 parts

Commit message: add fabrication files bottom board
Parts:
- added H8, H9: HOLE, MountingHole:MountingHole_3mm, symbol bottom-board-rescue:HOLE-local-components
Changed lines of the file:
@@
+	1    0    0    -1
+$EndComp
+$Comp
+L bottom-board-rescue:HOLE-local-components H?
+U 1 1 5DFE1600
+P 5100 1400
+AR Path="/5DFE1600" Ref="H?"  Part="1"
+AR Path="/55FC02AF/5DFE1600" Ref="H8"  Part="1"
+F 0 "H8" H 5100 1220 50  0000 C CNN
+F 1 "HOLE" H 5100 1570 50  0000 C CNN
+F 2 "MountingHole:MountingHole_3mm" H 5100 1400 60  0001 C CNN
+F 3 "" H 5100 1400 60  0000 C CNN
+	1    5100 1400
+	1    0    0    -1
+$EndComp
+$Comp
+L bottom-board-rescue:HOLE-local-components H?
+U 1 1 5DFE1606
+P 5450 1400
+AR Path="/5DFE1606" Ref="H?"  Part="1"
+AR Path="/55FC02AF/5DFE1606" Ref="H9"  Part="1"
+F 0 "H9" H 5450 1220 50  0000 C CNN
+F 1 "HOLE" H 5450 1570 50  0000 C CNN
+F 2 "MountingHole:MountingHole_3mm" H 5450 1400 60  0001 C CNN
+F 3 "" H 5450 1400 60  0000 C CNN
+	1    5450 1400
 	1    0    0    -1
 $EndComp
