File: bottom-board/usb.sch (KiCad schematic (older format))
At the start: 14 parts, among them P1 USB_B, P2 USB_A, U10 RT9742MNGJ5

Commit message: add fabrication files bottom board
Parts:
- R42: value 5k6 -> 5K6
Changed lines of the file:
@@
 P 2550 3350
 F 0 "R42" H 2600 3400 50  0000 L CNN
-F 1 "5k6" H 2600 3300 50  0000 L CNN
+F 1 "5K6" H 2600 3300 50  0000 L CNN
 F 2 "Resistor_SMD:R_0603_1608Metric" H 2550 3350 60  0001 C CNN
 F 3 "" H 2550 3350 60  0000 C CNN
