File: bottom-board/power.sch (KiCad schematic (older format))
At the start: 21 parts, among them U1 TS2596, U2 LD1117S50TR_SOT223

Commit message: add fabrication files bottom board
Parts:
- L2: value INDUCTOR -> 47UH 2A 135 MOHM
Changed lines of the file:
@@
 P 6700 4850
 F 0 "L2" H 6700 5065 50  0000 C CNN
-F 1 "INDUCTOR" H 6700 4974 50  0000 C CNN
+F 1 "47UH 2A 135 MOHM" H 6700 4974 50  0000 C CNN
 F 2 "Uno:SRN8040TA" H 6700 4850 50  0001 C CNN
 F 3 "https://www.digikey.com/product-detail/en/bourns-inc/SRN8040TA-470M/SRN8040TA-470MTR-ND/6155133" H 6700 4850 50  0001 C CNN

Commit message: reposistioned PSU filtering caps
Parts:
- C2, C6: footprint Capacitor_THT:CP_Radial_D13.0mm_P5.00mm -> Capacitor_THT:CP_Radial_D10.0mm_P5.00mm
- C3, C32: footprint Capacitor_SMD:CP_Elec_10x7.9 -> Capacitor_SMD:CP_Elec_8x10.5
Changed lines of the file:
@@
 F 0 "C6" H 5675 3150 50  0000 L CNN
 F 1 "2200uF" H 5675 2950 50  0000 L CNN
-F 2 "Capacitor_THT:CP_Radial_D13.0mm_P5.00mm" H 5688 2900 30  0001 C CNN
+F 2 "Capacitor_THT:CP_Radial_D10.0mm_P5.00mm" H 5688 2900 30  0001 C CNN
 F 3 "" H 5650 3050 60  0000 C CNN
 F 4 "	UUG1C222MNQ6MS" H 800 250 50  0001 C CNN "MPN"
@@
 F 0 "C2" H 4325 3150 50  0000 L CNN
 F 1 "2200uF" H 4325 2950 50  0000 L CNN
-F 2 "Capacitor_THT:CP_Radial_D13.0mm_P5.00mm" H 4338 2900 30  0001 C CNN
+F 2 "Capacitor_THT:CP_Radial_D10.0mm_P5.00mm" H 4338 2900 30  0001 C CNN
 F 3 "" H 4300 3050 60  0000 C CNN
 F 4 "	UUG1C222MNQ6MS" H 800 250 50  0001 C CNN "MPN"
@@
 F 0 "C3" H 4325 5050 50  0000 L CNN
 F 1 "470uF" H 4050 4850 50  0000 L CNN
-F 2 "Capacitor_SMD:CP_Elec_10x7.9" H 4338 4800 30  0001 C CNN
+F 2 "Capacitor_SMD:CP_Elec_8x10.5" H 4338 4800 30  0001 C CNN
 F 3 "" H 4300 4950 60  0000 C CNN
 F 4 "UWT1C471MNL1GS" H 800 2150 50  0001 C CNN "MPN"
@@
 F 0 "C32" H 7425 5200 50  0000 L CNN
 F 1 "470uF" H 7150 5000 50  0000 L CNN
-F 2 "Capacitor_SMD:CP_Elec_10x7.9" H 7438 4950 30  0001 C CNN
+F 2 "Capacitor_SMD:CP_Elec_8x10.5" H 7438 4950 30  0001 C CNN
 F 3 "" H 7400 5100 60  0000 C CNN
 F 4 "UWT1C471MNL1GS" H 3900 2300 50  0001 C CNN "MPN"
