File: bottom-board/PCB Source/bottom-board/audio-outputs.sch (KiCad schematic (older format))
At the start: 39 parts, among them P11 JACK_TRS_6PINS, P12 JACK_TRS_6PINS, U6 TL082, U7 TL082

Commit message: rev 0.0.3
Parts:
- removed C38: 10uF, Capacitor_SMD:C_0603_1608Metric, symbol bottom-board-rescue:C_Small
- removed C40, C47, C55: 10uF, Capacitor_SMD:CP_Elec_4x5.7, symbol bottom-board-rescue:CP_Small
- removed C56: 100uF, Capacitor_SMD:CP_Elec_6.3x7.7, symbol bottom-board-rescue:CP_Small
- removed FB5: Ferrite_Bead, Resistor_SMD:R_0603_1608Metric, symbol Device:Ferrite_Bead
- removed R70, R71, R72, R74, R76, R77: 10K, Resistor_SMD:R_0603_1608Metric, symbol Device:R_Small
- removed R80, R82, R84, R86: 33R, Resistor_SMD:R_0603_1608Metric, symbol Device:R_Small
- removed R81, R83: 22K 1%, Resistor_SMD:R_0603_1608Metric, symbol Device:R_Small
- removed R85, R87: 68R, Resistor_SMD:R_0603_1608Metric, symbol Device:R_Small
- added C40, C47, C55, C56, C90, C91: 100pF, Capacitor_SMD:C_0603_1608Metric, symbol bottom-board-rescue:C_Small
- added C74, C83, C84: 47uF, Capacitor_SMD:CP_Elec_5x5.4, symbol bottom-board-rescue:CP_Small
- added C88, C89: 10uF, Capacitor_SMD:CP_Elec_4x5.7, symbol bottom-board-rescue:CP_Small
- added D19, D20, D21, D22: BAT54S, Package_TO_SOT_SMD:SOT-23, symbol bottom-board-rescue:BAT54S-Diode
- added R102, R105, R106, R107, R108, R109, R86, R87: 150R, Resistor_SMD:R_0603_1608Metric, symbol bottom-board-rescue:R_Small-Device
- added R74, R76, R77, R80, R81, R82, R83, R84, R85, R98: 10K, Resistor_SMD:R_0603_1608Metric, symbol bottom-board-rescue:R_Small-Device
- added R8: 100R, Resistor_SMD:R_0603_1608Metric, symbol bottom-board-rescue:R_Small-Device
- C42: value 10uF -> 47uF; footprint Capacitor_SMD:CP_Elec_4x5.7 -> Capacitor_SMD:CP_Elec_5x5.4; MPN EEE-HB1C100R -> EDK476M016A9DAA
- C57: value 100uF -> 47uF; footprint Capacitor_SMD:CP_Elec_6.3x7.7 -> Capacitor_SMD:CP_Elec_5x5.4; MPN UWX1C101MCL1GB -> EDK476M016A9DAA
- P11, P12: symbol Connector:AudioJack3_Switch -> bottom-board-rescue:AudioJack3_Switch-Connector
- R73, R75, R78, R79: symbol Device:R_Small -> bottom-board-rescue:R_Small-Device
- TP8: symbol Connector:TestPoint -> bottom-board-rescue:TestPoint-Connector
- U6, U7: value TL082 -> OPA1678; symbol Amplifier_Operational:TL072 -> bottom-board-rescue:TL072-Amplifier_Operational; MPN TL082CDR -> OPA1678IDR
- U6, U7: value TL082 -> OPA1678; footprint (none) -> Package_SO:SOIC-8_3.9x4.9mm_P1.27mm; symbol Amplifier_Operational:TL072 -> bottom-board-rescue:TL072-Amplifier_Operational
Connections:
- net labels added: +10V, +5VA
- net labels removed: +12VA
- wire segments 126 -> 186
Other:
- note removed: "*** Output Gain ***\n\n"""\nOpAmps are configured to not make any gain, this can be adjusted\nfor but every dB of gain will be added to the noise floor as well\nMAX Gian:\nCodec: 0.65 * Va = 0.65 * 5 = 3.25Vp\n=1.15V RMS line level is 1.25V RMS\n""""
- note removed: "*** The outputs are not balanced ***\n\n"""\nThe Ring pin is actually a low impedance input, and any \nsignal on it is added to the output signal. This will make a\nbalanced input see only the signal, and provides exactly the\nsame level (and even ground loop compensation) to an \nunbalanced input.\n""""
- note removed: "Use feritte beads for EMI suppression and improved power supply decoupling"
- moved on the sheet: C46, R73, R75, R78, R79, R88, R89

Commit message: cleanup BOM lines
Parts:
- C41, C45: MPN CL10A106MQ8NNNC -> EMK107BBJ106MA-T
- R8: MPN RMCF0603JT100R -> RT0603DRD07100RL
- R88, R89: MPN CR0603-JW-104ELF -> RMCF0603JT100K
Changed lines of the file:
@@
 encoding utf-8
 Sheet 6 11
-Title "MOD Uno - Main Board"
-Date "2019-08-16"
-Rev "0.1"
+Title "MOD Dwarf - Main Board"
+Date "2021-04-07"
+Rev "1.2"
 Comp "MOD Devices GmbH"
-Comment1 "Uno Audio processing board"
-Comment2 "https://github.com/moddevices/hw-mod-uno"
+Comment1 "Dwarf Audio processing board"
+Comment2 "https://github.com/moddevices/hw-mod-dwarf"
 Comment3 "Inp Power: 12V 500mA"
 Comment4 "USB outp Power: 500mA"
@@
 F 2 "Capacitor_SMD:C_0603_1608Metric" H 2605 7080 60  0001 C CNN
 F 3 "" H 2605 7080 60  0000 C CNN
-F 4 "CL10A106MQ8NNNC" H -1845 5380 50  0001 C CNN "MPN"
+F 4 "EMK107BBJ106MA-T" H -1845 5380 50  0001 C CNN "MPN"
 	1    2605 7080
 	-1   0    0    1
@@
 F 2 "Capacitor_SMD:C_0603_1608Metric" H 3525 7070 60  0001 C CNN
 F 3 "" H 3525 7070 60  0000 C CNN
-F 4 "CL10A106MQ8NNNC" H -925 5370 50  0001 C CNN "MPN"
+F 4 "EMK107BBJ106MA-T" H -925 5370 50  0001 C CNN "MPN"
 	1    3525 7070
 	-1   0    0    1
@@
 F 2 "Resistor_SMD:R_0603_1608Metric" H 6245 2470 60  0001 C CNN
 F 3 "" H 6245 2470 60  0000 C CNN
-F 4 "CR0603-JW-104ELF" H 6245 2470 50  0001 C CNN "MPN"
+F 4 "RMCF0603JT100K" H 6245 2470 50  0001 C CNN "MPN"
 	1    6245 2470
 	-1   0    0    -1
@@
 F 2 "Resistor_SMD:R_0603_1608Metric" H 6315 4570 60  0001 C CNN
 F 3 "" H 6315 4570 60  0000 C CNN
-F 4 "CR0603-JW-104ELF" H 6315 4570 50  0001 C CNN "MPN"
+F 4 "RMCF0603JT100K" H 6315 4570 50  0001 C CNN "MPN"
 	1    6315 4570
 	-1   0    0    -1
@@
 F 2 "Resistor_SMD:R_0603_1608Metric" H 1115 6865 50  0001 C CNN
 F 3 "" H 1115 6865 50  0001 C CNN
-F 4 "RMCF0603JT100R" V 1115 6865 50  0001 C CNN "MPN"
+F 4 "RT0603DRD07100RL" V 1115 6865 50  0001 C CNN "MPN"
 	1    1115 6865
 	1    0    0    1
