File: bottom-board/PCB Source/bottom-board/control-chain.sch (KiCad schematic (older format))
At the start: 14 parts, among them P13 RJ45, U12 ISL83491

Commit message: rev 0.0.3
Parts:
- C54, C62: MPN C1608X7R1E104K080AA -> GCM188R71C104KA37D
- C61: footprint Capacitor_SMD:CP_Elec_5x5.3 -> Capacitor_SMD:CP_Elec_4x5.7; MPN UWX1E100MCL1GB -> EEE-HB1C100R
- P13: symbol Connector:RJ45 -> bottom-board-rescue:RJ45-Connector
- R57, R58: value 10k -> 10K; MPN RMCF0603JT10K0 -> RR0816P-103-D
Changed lines of the file:
@@
 F 2 "Capacitor_SMD:C_0603_1608Metric" H 3515 2560 60  0001 C CNN
 F 3 "" H 3515 2560 60  0000 C CNN
-F 4 "C1608X7R1E104K080AA" H -1335 810 50  0001 C CNN "MPN"
+F 4 "GCM188R71C104KA37D" H -1335 810 50  0001 C CNN "MPN"
 	1    3515 2560
 	0    -1   1    0
@@
 P 2665 2810
 F 0 "R57" H 2715 2860 50  0000 L CNN
-F 1 "10k" H 2715 2760 50  0000 L CNN
+F 1 "10K" H 2715 2760 50  0000 L CNN
 F 2 "Resistor_SMD:R_0603_1608Metric" H 2665 2810 60  0001 C CNN
-F 3 "" H 2665 2810 60  0000 C CNN
-F 4 "RMCF0603JT10K0" H -585 1510 50  0001 C CNN "MPN"
+F 3 "~" H 2665 2810 60  0000 C CNN
+F 4 "RR0816P-103-D" H -585 1510 50  0001 C CNN "MPN"
 	1    2665 2810
 	1    0    0    -1
@@
 P 2665 4010
 F 0 "R58" H 2715 4060 50  0000 L CNN
-F 1 "10k" H 2715 3960 50  0000 L CNN
+F 1 "10K" H 2715 3960 50  0000 L CNN
 F 2 "Resistor_SMD:R_0603_1608Metric" H 2665 4010 60  0001 C CNN
-F 3 "" H 2665 4010 60  0000 C CNN
-F 4 "RMCF0603JT10K0" H -585 2710 50  0001 C CNN "MPN"
+F 3 "~" H 2665 4010 60  0000 C CNN
+F 4 "RR0816P-103-D" H -585 2710 50  0001 C CNN "MPN"
 	1    2665 4010
 	1    0    0    -1
@@
 $EndComp
 $Comp
-L bottom-board-rescue:CP_Small C?
-U 1 1 5F5E8B0C
-P 7405 3510
-AR Path="/54F72FB8/5F5E8B0C" Ref="C?"  Part="1"
-AR Path="/54F72FB6/5F5E8B0C" Ref="C61"  Part="1"
-F 0 "C61" H 7455 3410 50  0000 L CNN
-F 1 "10uF" V 7455 3560 50  0000 L CNN
-F 2 "Capacitor_SMD:CP_Elec_5x5.3" H 7405 3510 60  0001 C CNN
-F 3 "" H 7405 3510 60  0000 C CNN
-F 4 "UWX1E100MCL1GB" H -345 -1440 50  0001 C CNN "MPN"
-	1    7405 3510
-	1    0    0    -1
-$EndComp
-$Comp
 L bottom-board-rescue:GNDD-power #PWR?
 U 1 1 5F5E8B12
@@
 F 2 "Capacitor_SMD:C_0603_1608Metric" H 7705 3510 60  0001 C CNN
 F 3 "" H 7705 3510 60  0000 C CNN
-F 4 "C1608X7R1E104K080AA" H -345 -1440 50  0001 C CNN "MPN"
+F 4 "GCM188R71C104KA37D" H -345 -1440 50  0001 C CNN "MPN"
 	1    7705 3510
 	1    0    0    -1
 $EndComp
 $Comp
-L Connector:RJ45 P?
+L bottom-board-rescue:RJ45-Connector P?
 U 1 1 5F5E8B3D
 P 8905 3210
@@
 Text Notes 5965 2660 0    60   ~ 0
 This port is NOT used for ethernet, but for a serial protocol that includes power over the RJ-45 connector
+$Comp
+L bottom-board-rescue:CP_Small C?
+U 1 1 5FAE2F8E
+P 7405 3510
+AR Path="/54F7244B/5FAE2F8E" Ref="C?"  Part="1"
+AR Path="/54F72B97/5FAE2F8E" Ref="C?"  Part="1"
+AR Path="/54F72C8D/5FAE2F8E" Ref="C?"  Part="1"
+AR Path="/54F72FB6/5FAE2F8E" Ref="C61"  Part="1"
+F 0 "C61" H 7475 3430 50  0000 L CNN
+F 1 "10uF" H 7475 3510 50  0000 L CNN
+F 2 "Capacitor_SMD:CP_Elec_4x5.7" H 7443 3360 30  0001 C CNN
+F 3 "" H 7405 3510 60  0000 C CNN
+F 4 "EEE-HB1C100R" H 3905 710 50  0001 C CNN "MPN"
+	1    7405 3510
+	1    0    0    -1
+$EndComp
 $EndSCHEMATC

Commit message: change design to 4 layer PCB
Parts:
- R59, R60, R61, R62: MPN ERJ-P6WJ560V -> CRGCQ0603F56R
Changed lines of the file:
@@
 F 2 "Resistor_SMD:R_0603_1608Metric" H 3965 3010 60  0001 C CNN
 F 3 "" H 3965 3010 60  0000 C CNN
-F 4 "ERJ-P6WJ560V" H -2035 810 50  0001 C CNN "MPN"
+F 4 "CRGCQ0603F56R" H -2035 810 50  0001 C CNN "MPN"
 	1    3965 3010
 	0    1    1    0
@@
 F 2 "Resistor_SMD:R_0603_1608Metric" H 3965 3210 60  0001 C CNN
 F 3 "" H 3965 3210 60  0000 C CNN
-F 4 "ERJ-P6WJ560V" H -2035 810 50  0001 C CNN "MPN"
+F 4 "CRGCQ0603F56R" H -2035 810 50  0001 C CNN "MPN"
 	1    3965 3210
 	0    1    1    0
@@
 F 2 "Resistor_SMD:R_0603_1608Metric" H 4215 3510 60  0001 C CNN
 F 3 "" H 4215 3510 60  0000 C CNN
-F 4 "ERJ-P6WJ560V" H -2035 810 50  0001 C CNN "MPN"
+F 4 "CRGCQ0603F56R" H -2035 810 50  0001 C CNN "MPN"
 	1    4215 3510
 	0    1    1    0
@@
 F 2 "Resistor_SMD:R_0603_1608Metric" H 4215 3710 60  0001 C CNN
 F 3 "" H 4215 3710 60  0000 C CNN
-F 4 "ERJ-P6WJ560V" H -2035 810 50  0001 C CNN "MPN"
+F 4 "CRGCQ0603F56R" H -2035 810 50  0001 C CNN "MPN"
 	1    4215 3710
 	0    1    1    0

Commit message: cleanup BOM lines
Parts:
- R55, R56, R63: MPN RMCF0603JT100R -> RT0603DRD07100RL
Changed lines of the file:
@@
 encoding utf-8
 Sheet 9 11
-Title "MOD Uno - Main Board"
-Date "2019-08-16"
-Rev "0.1"
+Title "MOD Dwarf - Main Board"
+Date "2021-04-07"
+Rev "1.2"
 Comp "MOD Devices GmbH"
-Comment1 "Uno Audio processing board"
-Comment2 "https://github.com/moddevices/hw-mod-uno"
+Comment1 "Dwarf Audio processing board"
+Comment2 "https://github.com/moddevices/hw-mod-dwarf"
 Comment3 "Inp Power: 12V 500mA"
 Comment4 "USB outp Power: 500mA"
@@
 F 2 "Resistor_SMD:R_0603_1608Metric" H 4515 3110 60  0001 C CNN
 F 3 "" H 4515 3110 60  0000 C CNN
-F 4 "RMCF0603JT100R" H -2035 810 50  0001 C CNN "MPN"
+F 4 "RT0603DRD07100RL" H -2035 810 50  0001 C CNN "MPN"
 	1    4515 3110
 	1    0    0    -1
@@
 F 2 "Resistor_SMD:R_0603_1608Metric" H 2515 3110 60  0001 C CNN
 F 3 "" H 2515 3110 60  0000 C CNN
-F 4 "RMCF0603JT100R" H -2035 810 50  0001 C CNN "MPN"
+F 4 "RT0603DRD07100RL" H -2035 810 50  0001 C CNN "MPN"
 	1    2515 3110
 	0    1    1    0
@@
 F 2 "Resistor_SMD:R_0603_1608Metric" H 2465 3610 60  0001 C CNN
 F 3 "" H 2465 3610 60  0000 C CNN
-F 4 "RMCF0603JT100R" H -2085 810 50  0001 C CNN "MPN"
+F 4 "RT0603DRD07100RL" H -2085 810 50  0001 C CNN "MPN"
 	1    2465 3610
 	0    1    1    0
