File: bottom-board/PCB Source/bottom-board/control-chain.sch (KiCad schematic (older format))
At the start: 14 parts, among them P13 RJ45, U12 ISL83491

Commit message: change JFET MPN
Parts:
- U12: MPN ISL3176EIBZ -> ISL83491IBZ
Changed lines of the file:
@@
 F 2 "Package_SO:SOIC-14_3.9x8.7mm_P1.27mm" H 3265 3410 50  0001 C CIN
 F 3 "" H 3265 3410 60  0000 C CNN
-F 4 "ISL3176EIBZ" H -2035 810 50  0001 C CNN "MPN"
+F 4 "ISL83491IBZ" H -2035 810 50  0001 C CNN "MPN"
 	1    3265 3410
 	1    0    0    -1

Commit message: change input bias 5->6V, reduce harmonics
Parts:
- U12: MPN ISL83491IBZ -> ISL3176EIBZ
Changed lines of the file:
@@
 F 2 "Package_SO:SOIC-14_3.9x8.7mm_P1.27mm" H 3265 3410 50  0001 C CIN
 F 3 "" H 3265 3410 60  0000 C CNN
-F 4 "ISL83491IBZ" H -2035 810 50  0001 C CNN "MPN"
+F 4 "ISL3176EIBZ" H -2035 810 50  0001 C CNN "MPN"
 	1    3265 3410
 	1    0    0    -1
