File: bottom-board/PCB Source/bottom-board/midi.sch (KiCad schematic (older format))
At the start: 12 parts, among them P6 AudioJack3, P7 AudioJack3, Q12 2N7002, Q13 2N7002, U11 6N137S

Commit message: rev 0.0.3
Parts:
- added C82: 100nF, Capacitor_SMD:C_0603_1608Metric, symbol bottom-board-rescue:C_Small
- added D12: BAT54S, Package_TO_SOT_SMD:SOT-23, symbol bottom-board-rescue:BAT54S-Diode
- D15, D16: footprint Diode_SMD:D_SOD-523 -> Diode_SMD:D_SOD-323; symbol Diode:1N4148 -> bottom-board-rescue:1N4148-Diode; MPN 1N4148X-TP -> 1N4148WS
- P6, P7: symbol Connector:AudioJack3 -> bottom-board-rescue:AudioJack3-Connector
- R51, R52: value 10k -> 10K; MPN RMCF0603JT10K0 -> RR0816P-103-D
Connections:
- wire segments 34 -> 40
Changed lines of the file:
@@
 P 7950 3350
 F 0 "R51" H 8000 3400 50  0000 L CNN
-F 1 "10k" H 8000 3300 50  0000 L CNN
+F 1 "10K" H 8000 3300 50  0000 L CNN
 F 2 "Resistor_SMD:R_0603_1608Metric" H 7950 3350 60  0001 C CNN
-F 3 "" H 7950 3350 60  0000 C CNN
-F 4 "RMCF0603JT10K0" H 350 0   50  0001 C CNN "MPN"
+F 3 "~" H 7950 3350 60  0000 C CNN
+F 4 "RR0816P-103-D" H 350 0   50  0001 C CNN "MPN"
 	1    7950 3350
 	1    0    0    -1
@@
 P 8500 3650
 F 0 "R52" H 8550 3700 50  0000 L CNN
-F 1 "10k" H 8550 3600 50  0000 L CNN
+F 1 "10K" H 8550 3600 50  0000 L CNN
 F 2 "Resistor_SMD:R_0603_1608Metric" H 8500 3650 60  0001 C CNN
-F 3 "" H 8500 3650 60  0000 C CNN
-F 4 "RMCF0603JT10K0" H 150 0   50  0001 C CNN "MPN"
+F 3 "~" H 8500 3650 60  0000 C CNN
+F 4 "RR0816P-103-D" H 150 0   50  0001 C CNN "MPN"
 	1    8500 3650
 	1    0    0    -1
@@
 	8500 3850 8500 3950
 $Comp
-L Connector:AudioJack3 P6
+L bottom-board-rescue:AudioJack3-Connector P6
 U 1 1 5D15D509
 P 2345 3445
@@
 NoConn ~ 2445 3645
 $Comp
-L Diode:1N4148 D?
+L bottom-board-rescue:1N4148-Diode D?
 U 1 1 5D5B626A
 P 3220 3920
@@
 F 0 "D15" V 3220 3830 50  0000 R CNN
 F 1 "1N4148" V 3305 3850 50  0000 R CNN
-F 2 "Diode_SMD:D_SOD-523" H 3220 3745 50  0001 C CNN
+F 2 "Diode_SMD:D_SOD-323" H 3220 3745 50  0001 C CNN
 F 3 "https://assets.nexperia.com/documents/data-sheet/1N4148_1N4448.pdf" H 3220 3920 50  0001 C CNN
-F 4 "1N4148X-TP" V 3220 3920 50  0001 C CNN "MPN"
+F 4 "1N4148WS" V 3220 3920 50  0001 C CNN "MPN"
 	1    3220 3920
 	0    1    1    0
@@
 	3220 3720 3520 3720
 $Comp
-L Diode:1N4148 D?
+L bottom-board-rescue:1N4148-Diode D?
 U 1 1 5D5BA7F0
 P 4370 3920
@@
 F 0 "D16" H 4430 4035 50  0000 R CNN
 F 1 "1N4148" H 4505 3835 50  0000 R CNN
-F 2 "Diode_SMD:D_SOD-523" H 4370 3745 50  0001 C CNN
+F 2 "Diode_SMD:D_SOD-323" H 4370 3745 50  0001 C CNN
 F 3 "https://assets.nexperia.com/documents/data-sheet/1N4148_1N4448.pdf" H 4370 3920 50  0001 C CNN
-F 4 "1N4148X-TP" V 4370 3920 50  0001 C CNN "MPN"
+F 4 "1N4148WS" V 4370 3920 50  0001 C CNN "MPN"
 	1    4370 3920
 	1    0    0    -1
@@
 	3220 4205 2245 4205
 Wire Wire Line
-	4230 3535 4230 3620
-Wire Wire Line
 	4120 3620 4230 3620
 Wire Wire Line
 	4565 3920 4520 3920
 $Comp
-L Connector:AudioJack3 P7
+L bottom-board-rescue:AudioJack3-Connector P7
 U 1 1 5D15C2EF
 P 7025 3075
@@
 Wire Notes Line
 	5450 2750 5450 4695
+$Comp
+L bottom-board-rescue:C_Small C?
+U 1 1 5FC6848F
+P 4445 3615
+AR Path="/54F72B97/5FC6848F" Ref="C?"  Part="1"
+AR Path="/54F72C8D/5FC6848F" Ref="C?"  Part="1"
+AR Path="/54F72FB4/5FC6848F" Ref="C82"  Part="1"
+F 0 "C82" H 4340 3545 50  0000 L CNN
+F 1 "100nF" H 4190 3720 50  0000 L CNN
+F 2 "Capacitor_SMD:C_0603_1608Metric" H 4445 3615 60  0001 C CNN
+F 3 "" H 4445 3615 60  0000 C CNN
+F 4 "GCM188R71C104KA37D" H -855 -1735 50  0001 C CNN "MPN"
+	1    4445 3615
+	0    1    1    0
+$EndComp
+Wire Wire Line
+	4345 3615 4230 3615
+Wire Wire Line
+	4230 3535 4230 3615
+Connection ~ 4230 3615
+Wire Wire Line
+	4230 3615 4230 3620
+$Comp
+L bottom-board-rescue:GNDD-power #PWR0264
+U 1 1 5FC72014
+P 4650 3615
+F 0 "#PWR0264" H 4650 3365 50  0001 C CNN
+F 1 "GNDD" H 4650 3465 50  0000 C CNN
+F 2 "" H 4650 3615 60  0000 C CNN
+F 3 "" H 4650 3615 60  0000 C CNN
+	1    4650 3615
+	0    -1   -1   0
+$EndComp
+Wire Wire Line
+	4650 3615 4545 3615
+$Comp
+L bottom-board-rescue:BAT54S-Diode D?
+U 1 1 5FCD8EEA
+P 7025 3750
+AR Path="/54F72B97/5FCD8EEA" Ref="D?"  Part="1"
+AR Path="/54F72C8D/5FCD8EEA" Ref="D?"  Part="1"
+AR Path="/54F72FB4/5FCD8EEA" Ref="D12"  Part="1"
+F 0 "D12" H 6815 3625 50  0000 L CNN
+F 1 "BAT54S" H 6840 3880 50  0000 L CNN
+F 2 "Package_TO_SOT_SMD:SOT-23" H 7100 3875 50  0001 L CNN
+F 3 "https://www.diodes.com/assets/Datasheets/ds11005.pdf" H 6905 3750 50  0001 C CNN
+F 4 "BAT54SFILM" V 7025 3750 50  0001 C CNN "MPN"
+	1    7025 3750
+	1    0    0    1
+$EndComp
+Connection ~ 7025 3550
+$Comp
+L bottom-board-rescue:+5V-power #PWR0265
+U 1 1 5FCE0A00
+P 7360 3750
+F 0 "#PWR0265" H 7360 3600 50  0001 C CNN
+F 1 "+5V" H 7360 3890 50  0000 C CNN
+F 2 "" H 7360 3750 60  0000 C CNN
+F 3 "" H 7360 3750 60  0000 C CNN
+	1    7360 3750
+	1    0    0    -1
+$EndComp
+$Comp
+L bottom-board-rescue:GNDD-power #PWR0266
+U 1 1 5FCE18B6
+P 6680 3760
+F 0 "#PWR0266" H 6680 3510 50  0001 C CNN
+F 1 "GNDD" H 6680 3610 50  0000 C CNN
+F 2 "" H 6680 3760 60  0000 C CNN
+F 3 "" H 6680 3760 60  0000 C CNN
+	1    6680 3760
+	1    0    0    -1
+$EndComp
+Wire Wire Line
+	6680 3760 6680 3750
+Wire Wire Line
+	6680 3750 6725 3750
+Wire Wire Line
+	7325 3750 7360 3750
 $EndSCHEMATC

Commit message: change design to 4 layer PCB
Parts:
- R47, R49, R50: MPN RL73N1JR22JTD -> RC0603FR-07220RL
- U11: footprint Package_DIP:DIP-8_W7.62mm_SMDSocket_SmallPads -> Uno:6N137S
Changed lines of the file:
@@
 F 2 "Resistor_SMD:R_0603_1608Metric" H 6665 3335 60  0001 C CNN
 F 3 "" H 6665 3335 60  0000 C CNN
-F 4 "RL73N1JR22JTD" H 365 -15 50  0001 C CNN "MPN"
+F 4 "RC0603FR-07220RL" H 365 -15 50  0001 C CNN "MPN"
 	1    6665 3335
 	0    1    1    0
@@
 F 2 "Resistor_SMD:R_0603_1608Metric" H 7700 3550 60  0001 C CNN
 F 3 "" H 7700 3550 60  0000 C CNN
-F 4 "RL73N1JR22JTD" H 350 0   50  0001 C CNN "MPN"
+F 4 "RC0603FR-07220RL" H 350 0   50  0001 C CNN "MPN"
 	1    7700 3550
 	0    -1   -1   0
@@
 F 0 "U11" H 3570 3520 50  0000 L CNN
 F 1 "6N137S" H 3820 3520 50  0000 L CNN
-F 2 "Package_DIP:DIP-8_W7.62mm_SMDSocket_SmallPads" H 3620 3520 50  0001 L CIN
+F 2 "Uno:6N137S" H 3620 3520 50  0001 L CIN
 F 3 "" H 3820 3820 50  0000 L CNN
 F 4 "6N137S" H 170 170 50  0001 C CNN "MPN"
@@
 F 2 "Resistor_SMD:R_0603_1608Metric" H 2920 3720 60  0001 C CNN
 F 3 "" H 2920 3720 60  0000 C CNN
-F 4 "RL73N1JR22JTD" H -3380 370 50  0001 C CNN "MPN"
+F 4 "RC0603FR-07220RL" H -3380 370 50  0001 C CNN "MPN"
 	1    2920 3720
 	0    -1   -1   0

Commit message: minor cleanup
Connections:
- net at R49.1: now also P7.R; no longer P7.T
- net at D12.3, R50.1: now also P7.T; no longer P7.R
Other:
- moved on the sheet: P7, R49
Changed lines of the file:
@@
 L bottom-board-rescue:R_Small R49
 U 1 1 550EE5CB
-P 6665 3335
-F 0 "R49" V 6590 3265 50  0000 L CNN
-F 1 "220R" V 6740 3240 50  0000 L CNN
-F 2 "Resistor_SMD:R_0603_1608Metric" H 6665 3335 60  0001 C CNN
-F 3 "" H 6665 3335 60  0000 C CNN
-F 4 "RC0603FR-07220RL" H 365 -15 50  0001 C CNN "MPN"
-	1    6665 3335
-	0    1    1    0
+P 7205 3440
+F 0 "R49" V 7130 3370 50  0000 L CNN
+F 1 "220R" V 7280 3345 50  0000 L CNN
+F 2 "Resistor_SMD:R_0603_1608Metric" H 7205 3440 60  0001 C CNN
+F 3 "" H 7205 3440 60  0000 C CNN
+F 4 "RC0603FR-07220RL" H 905 90  50  0001 C CNN "MPN"
+	1    7205 3440
+	0    -1   -1   0
 $EndComp
 $Comp
@@
 L bottom-board-rescue:GNDD-power #PWR0185
 U 1 1 550D24C3
-P 7125 3320
-F 0 "#PWR0185" H 7125 3070 50  0001 C CNN
-F 1 "GNDD" H 7150 3185 50  0000 C CNN
-F 2 "" H 7125 3320 60  0000 C CNN
-F 3 "" H 7125 3320 60  0000 C CNN
-	1    7125 3320
-	1    0    0    -1
+P 7040 3270
+F 0 "#PWR0185" H 7040 3020 50  0001 C CNN
+F 1 "GNDD" H 7065 3135 50  0000 C CNN
+F 2 "" H 7040 3270 60  0000 C CNN
+F 3 "" H 7040 3270 60  0000 C CNN
+	1    7040 3270
+	0    -1   -1   0
 $EndComp
 $Comp
@@
 L bottom-board-rescue:+5V-power #PWR0189
 U 1 1 550D42BC
-P 6515 3335
-F 0 "#PWR0189" H 6515 3185 50  0001 C CNN
-F 1 "+5V" H 6515 3475 50  0000 C CNN
-F 2 "" H 6515 3335 60  0000 C CNN
-F 3 "" H 6515 3335 60  0000 C CNN
-	1    6515 3335
-	0    -1   -1   0
+P 7355 3440
+F 0 "#PWR0189" H 7355 3290 50  0001 C CNN
+F 1 "+5V" H 7355 3580 50  0000 C CNN
+F 2 "" H 7355 3440 60  0000 C CNN
+F 3 "" H 7355 3440 60  0000 C CNN
+	1    7355 3440
+	0    1    1    0
 $EndComp
 $Comp
@@
 	5850 2750 9950 2750
 Wire Wire Line
-	6565 3335 6515 3335
+	7305 3440 7355 3440
 Wire Wire Line
 	7950 3200 7950 3250
@@
 Wire Wire Line
 	8500 3850 8500 3950
-$Comp
-L bottom-board-rescue:AudioJack3-Connector P6
-U 1 1 5D15D509
-P 2345 3445
-F 0 "P6" V 2373 3215 50  0000 R CNN
-F 1 "AudioJack3" V 2045 3595 50  0000 R CNN
-F 2 "Connector_Audio:Jack_3.5mm_CUI_SJ-3523-SMT_Horizontal" H 2345 3445 50  0001 C CNN
-F 3 "~" H 2345 3445 50  0001 C CNN
-F 4 "SJ-3523-SMT-TR" V 2345 3445 50  0001 C CNN "MPN"
-	1    2345 3445
-	0    1    1    0
-$EndComp
-NoConn ~ 2445 3645
 $Comp
 L bottom-board-rescue:1N4148-Diode D?
@@
 $EndComp
 Wire Wire Line
-	2820 3720 2345 3720
-Wire Wire Line
-	2345 3720 2345 3645
-Wire Wire Line
-	3320 4205 3220 4205
-Wire Wire Line
-	2245 4205 2245 3645
-Wire Wire Line
-	3320 3920 3320 4205
-Wire Wire Line
-	3220 4070 3220 4205
-Connection ~ 3220 4205
-Wire Wire Line
-	3220 4205 2245 4205
-Wire Wire Line
 	4120 3620 4230 3620
 Wire Wire Line
@@
 L bottom-board-rescue:AudioJack3-Connector P7
 U 1 1 5D15C2EF
-P 7025 3075
-F 0 "P7" V 6961 3263 50  0000 L CNN
-F 1 "AudioJack3" V 7052 3263 50  0000 L CNN
-F 2 "Connector_Audio:Jack_3.5mm_CUI_SJ-3523-SMT_Horizontal" H 7025 3075 50  0001 C CNN
-F 3 "~" H 7025 3075 50  0001 C CNN
-F 4 "SJ-3523-SMT-TR" V 7025 3075 50  0001 C CNN "MPN"
-	1    7025 3075
+P 6940 3025
+F 0 "P7" V 6876 3213 50  0000 L CNN
+F 1 "AudioJack3" V 6967 3213 50  0000 L CNN
+F 2 "Connector_Audio:Jack_3.5mm_CUI_SJ-3523-SMT_Horizontal" H 6940 3025 50  0001 C CNN
+F 3 "~" H 6940 3025 50  0001 C CNN
+F 4 "SJ-3523-SMT-TR" V 6940 3025 50  0001 C CNN "MPN"
+	1    6940 3025
 	0    1    1    0
 $EndComp
@@
 	7600 3550 7025 3550
 Wire Wire Line
-	7025 3550 7025 3275
-Wire Wire Line
-	7125 3320 7125 3275
-Wire Wire Line
-	6925 3335 6925 3275
-Wire Wire Line
-	6765 3335 6925 3335
+	7040 3270 7040 3225
 Wire Notes Line
 	5450 4695 1600 4695
@@
 	1    0    0    1
 $EndComp
-Connection ~ 7025 3550
 $Comp
 L bottom-board-rescue:+5V-power #PWR0265
@@
 Wire Wire Line
 	7325 3750 7360 3750
+Wire Wire Line
+	3320 3920 3320 4205
+Wire Wire Line
+	3320 4205 3220 4205
+Wire Wire Line
+	3220 4070 3220 4205
+NoConn ~ 2445 3645
+$Comp
+L bottom-board-rescue:AudioJack3-Connector P6
+U 1 1 5D15D509
+P 2345 3445
+F 0 "P6" V 2373 3215 50  0000 R CNN
+F 1 "AudioJack3" V 2045 3595 50  0000 R CNN
+F 2 "Connector_Audio:Jack_3.5mm_CUI_SJ-3523-SMT_Horizontal" H 2345 3445 50  0001 C CNN
+F 3 "~" H 2345 3445 50  0001 C CNN
+F 4 "SJ-3523-SMT-TR" V 2345 3445 50  0001 C CNN "MPN"
+	1    2345 3445
+	0    1    1    0
+$EndComp
+Connection ~ 3220 4205
+Wire Wire Line
+	3220 4205 2245 4205
+Wire Wire Line
+	2245 4205 2245 3645
+Wire Wire Line
+	2345 3720 2345 3645
+Wire Wire Line
+	2820 3720 2345 3720
+Wire Wire Line
+	6940 3225 6940 3440
+Wire Wire Line
+	6940 3440 7105 3440
+Wire Wire Line
+	6840 3225 6840 3550
+Wire Wire Line
+	6840 3550 7025 3550
+Connection ~ 7025 3550
 $EndSCHEMATC
