File: bottom-board/PCB Source/bottom-board/usb.sch (KiCad schematic (older format))
At the start: 17 parts, among them P1 USB_B, P2 USB_A, U10 RT9742MNGJ5

Commit message: rev 0.0.3
Parts:
- removed FB6, FB7, FB8, FB9: Ferrite_Bead, Resistor_SMD:R_0603_1608Metric, symbol Device:Ferrite_Bead
- added C92, C93: 1nF, Capacitor_SMD:C_0603_1608Metric, symbol bottom-board-rescue:C_Small
- added R16, R48: 1M 1%, Resistor_SMD:R_0603_1608Metric, symbol bottom-board-rescue:R_Small-Device
- C48, C50, C51, C52: MPN C1608X7R1E104K080AA -> GCM188R71C104KA37D
- R42: value 5K6 -> 10K; MPN RMCF0603JT5K60 -> RR0816P-103-D
- R43: value 10k -> 15K
- R46: value 10k -> 10K; MPN RMCF0603JT10K0 -> RR0816P-103-D
Connections:
- wire segments 91 -> 101
Other:
- note removed: "Isolate USB in terms of EMI, also soften the data ramp."
- note removed: "No beads/filtering needed here, as most devices will be powered by the main system"
- note removed: "Not all beads are needed, prototype which ones are worthwhile to keep"
Changed lines of the file:
@@
 P 2160 3640
 F 0 "R42" H 2210 3690 50  0000 L CNN
-F 1 "5K6" H 2210 3590 50  0000 L CNN
+F 1 "10K" H 2210 3590 50  0000 L CNN
 F 2 "Resistor_SMD:R_0603_1608Metric" H 2160 3640 60  0001 C CNN
-F 3 "" H 2160 3640 60  0000 C CNN
-F 4 "RMCF0603JT5K60" H -40 240 50  0001 C CNN "MPN"
+F 3 "~" H 2160 3640 60  0000 C CNN
+F 4 "RR0816P-103-D" H 2160 3640 50  0001 C CNN "MPN"
 	1    2160 3640
 	1    0    0    -1
@@
 P 2160 3940
 F 0 "R43" H 2210 3990 50  0000 L CNN
-F 1 "10k" H 2210 3890 50  0000 L CNN
+F 1 "15K" H 2210 3890 50  0000 L CNN
 F 2 "Resistor_SMD:R_0603_1608Metric" H 2160 3940 60  0001 C CNN
 F 3 "" H 2160 3940 60  0000 C CNN
@@
 F 2 "Capacitor_SMD:C_0603_1608Metric" H 1910 3940 60  0001 C CNN
 F 3 "" H 1910 3940 60  0000 C CNN
-F 4 "C1608X7R1E104K080AA" H -40 240 50  0001 C CNN "MPN"
+F 4 "GCM188R71C104KA37D" H -40 240 50  0001 C CNN "MPN"
 	1    1910 3940
 	1    0    0    -1
@@
 F 2 "Capacitor_SMD:C_0603_1608Metric" H 4750 3600 60  0001 C CNN
 F 3 "" H 4750 3600 60  0000 C CNN
-F 4 "C1608X7R1E104K080AA" H -100 -50 50  0001 C CNN "MPN"
+F 4 "GCM188R71C104KA37D" H -100 -50 50  0001 C CNN "MPN"
 	1    4750 3600
 	-1   0    0    1
@@
 L bottom-board-rescue:GNDD-power #PWR0179
 U 1 1 550A73CA
-P 9350 2750
-F 0 "#PWR0179" H 9350 2500 50  0001 C CNN
-F 1 "GNDD" H 9350 2600 50  0000 C CNN
-F 2 "" H 9350 2750 60  0000 C CNN
-F 3 "" H 9350 2750 60  0000 C CNN
-	1    9350 2750
-	1    0    0    -1
+P 9635 2650
+F 0 "#PWR0179" H 9635 2400 50  0001 C CNN
+F 1 "GNDD" H 9635 2500 50  0000 C CNN
+F 2 "" H 9635 2650 60  0000 C CNN
+F 3 "" H 9635 2650 60  0000 C CNN
+	1    9635 2650
+	0    -1   -1   0
 $EndComp
 $Comp
@@
 P 7200 3800
 F 0 "R46" H 7250 3850 50  0000 L CNN
-F 1 "10k" H 7250 3750 50  0000 L CNN
+F 1 "10K" H 7250 3750 50  0000 L CNN
 F 2 "Resistor_SMD:R_0603_1608Metric" H 7200 3800 60  0001 C CNN
-F 3 "" H 7200 3800 60  0000 C CNN
-F 4 "RMCF0603JT10K0" H 250 0   50  0001 C CNN "MPN"
+F 3 "~" H 7200 3800 60  0000 C CNN
+F 4 "RR0816P-103-D" H 250 0   50  0001 C CNN "MPN"
 	1    7200 3800
 	1    0    0    -1
@@
 F 2 "Capacitor_SMD:C_0603_1608Metric" H 7500 3100 60  0001 C CNN
 F 3 "" H 7500 3100 60  0000 C CNN
-F 4 "C1608X7R1E104K080AA" H 250 0   50  0001 C CNN "MPN"
+F 4 "GCM188R71C104KA37D" H 250 0   50  0001 C CNN "MPN"
 	1    7500 3100
 	0    -1   -1   0
@@
 F 2 "Capacitor_SMD:C_0603_1608Metric" H 10400 3650 60  0001 C CNN
 F 3 "" H 10400 3650 60  0000 C CNN
-F 4 "C1608X7R1E104K080AA" H 250 0   50  0001 C CNN "MPN"
+F 4 "GCM188R71C104KA37D" H 250 0   50  0001 C CNN "MPN"
 	1    10400 3650
 	-1   0    0    1
@@
 Wire Wire Line
 	8750 3050 8750 3450
-Wire Wire Line
-	9250 2650 9350 2650
-Wire Wire Line
-	9350 2650 9350 2750
 Connection ~ 4750 3800
 Connection ~ 7250 3100
@@
 Wire Wire Line
 	9050 3050 9050 3200
-Wire Wire Line
-	2685 2315 2585 2315
 $Comp
 L bottom-board-rescue:GNDD-power #PWR0175
 U 1 1 5509E7DC
-P 2685 2315
-F 0 "#PWR0175" H 2685 2065 50  0001 C CNN
-F 1 "GNDD" H 2685 2165 50  0000 C CNN
-F 2 "" H 2685 2315 60  0000 C CNN
-F 3 "" H 2685 2315 60  0000 C CNN
-	1    2685 2315
+P 2965 2315
+F 0 "#PWR0175" H 2965 2065 50  0001 C CNN
+F 1 "GNDD" H 2965 2165 50  0000 C CNN
+F 2 "" H 2965 2315 60  0000 C CNN
+F 3 "" H 2965 2315 60  0000 C CNN
+	1    2965 2315
 	0    -1   -1   0
 $EndComp
-$Comp
-L Device:Ferrite_Bead FB?
-U 1 1 5F542396
-P 2085 2905
-AR Path="/54F72B97/5F542396" Ref="FB?"  Part="1"
-AR Path="/54F72FB2/5F542396" Ref="FB6"  Part="1"
-F 0 "FB6" H 1825 2875 50  0000 L CNN
-F 1 "Ferrite_Bead" H 1495 3160 50  0000 L CNN
-F 2 "Resistor_SMD:R_0603_1608Metric" V 2015 2905 50  0001 C CNN
-F 3 "~" H 2085 2905 50  0001 C CNN
-F 4 "BLM18HD102SH1D" H 2085 2905 50  0001 C CNN "MPN"
-	1    2085 2905
-	1    0    0    -1
-$EndComp
-$Comp
-L Device:Ferrite_Bead FB?
-U 1 1 5F543B98
-P 2185 3145
-AR Path="/54F72B97/5F543B98" Ref="FB?"  Part="1"
-AR Path="/54F72FB2/5F543B98" Ref="FB7"  Part="1"
-F 0 "FB7" H 1930 3160 50  0000 L CNN
-F 1 "Ferrite_Bead" H 1505 3500 50  0000 L CNN
-F 2 "Resistor_SMD:R_0603_1608Metric" V 2115 3145 50  0001 C CNN
-F 3 "~" H 2185 3145 50  0001 C CNN
-F 4 "BLM18HD102SH1D" H 2185 3145 50  0001 C CNN "MPN"
-	1    2185 3145
-	1    0    0    -1
-$EndComp
-Wire Wire Line
-	2085 2715 2085 2755
-Wire Wire Line
-	2185 2715 2185 2995
-$Comp
-L Device:Ferrite_Bead FB?
-U 1 1 5F54E813
-P 2285 2900
-AR Path="/54F72B97/5F54E813" Ref="FB?"  Part="1"
-AR Path="/54F72FB2/5F54E813" Ref="FB8"  Part="1"
-F 0 "FB8" H 2415 2880 50  0000 L CNN
-F 1 "Ferrite_Bead" H 1500 3080 50  0000 L CNN
-F 2 "Resistor_SMD:R_0603_1608Metric" V 2215 2900 50  0001 C CNN
-F 3 "~" H 2285 2900 50  0001 C CNN
-F 4 "BLM18HD102SH1D" H 2285 2900 50  0001 C CNN "MPN"
-	1    2285 2900
-	1    0    0    -1
-$EndComp
-$Comp
-L Device:Ferrite_Bead FB?
-U 1 1 5F550C38
-P 2385 3150
-AR Path="/54F72B97/5F550C38" Ref="FB?"  Part="1"
-AR Path="/54F72FB2/5F550C38" Ref="FB9"  Part="1"
-F 0 "FB9" H 2515 3140 50  0000 L CNN
-F 1 "Ferrite_Bead" H 1495 3715 50  0000 L CNN
-F 2 "Resistor_SMD:R_0603_1608Metric" V 2315 3150 50  0001 C CNN
-F 3 "~" H 2385 3150 50  0001 C CNN
-F 4 "BLM18HD102SH1D" H 2385 3150 50  0001 C CNN "MPN"
-	1    2385 3150
-	1    0    0    -1
-$EndComp
-Wire Wire Line
-	2385 2715 2385 3000
-Wire Wire Line
-	2285 2715 2285 2750
 Wire Wire Line
 	2085 3410 2290 3410
 Wire Wire Line
 	2290 3410 2290 3490
-Wire Wire Line
-	2085 3055 2085 3410
 Connection ~ 2290 3490
 Wire Wire Line
@@
 Connection ~ 2290 3410
 Wire Wire Line
-	2185 3295 2185 3380
-Wire Wire Line
 	2185 3380 2720 3380
 Wire Wire Line
@@
 Wire Wire Line
 	2720 4200 3600 4200
-Wire Wire Line
-	2285 3050 2285 3365
 Wire Wire Line
 	2285 3365 2735 3365
@@
 	0    -1   -1   0
 $EndComp
-Text Notes 2605 2845 0    60   ~ 0
-Isolate USB in terms of EMI, also soften the data ramp.
-Text Notes 1405 2125 0    60   ~ 0
-Not all beads are needed, prototype which ones are worthwhile to keep
-Text Notes 6320 2130 0    60   ~ 0
-No beads/filtering needed here, as most devices will be powered by the main system
+Wire Wire Line
+	2185 2715 2185 3380
+Wire Wire Line
+	2285 2715 2285 3365
+Wire Wire Line
+	2085 2715 2085 3410
+Wire Wire Line
+	2385 2715 2385 3300
+$Comp
+L bottom-board-rescue:C_Small C?
+U 1 1 5F880017
+P 2775 2315
+AR Path="/54F725AE/5F880017" Ref="C?"  Part="1"
+AR Path="/54F72FB2/5F880017" Ref="C92"  Part="1"
+F 0 "C92" V 2825 2365 50  0000 L CNN
+F 1 "1nF" V 2725 2365 50  0000 L CNN
+F 2 "Capacitor_SMD:C_0603_1608Metric" H 2775 2315 60  0001 C CNN
+F 3 "" H 2775 2315 60  0000 C CNN
+F 4 "C0603X7R500-103KNP" H -8125 215 50  0001 C CNN "MPN"
+	1    2775 2315
+	0    1    1    0
+$EndComp
+$Comp
+L bottom-board-rescue:R_Small-Device R?
+U 1 1 5F88C44B
+P 2790 2450
+AR Path="/54F72C8D/5F88C44B" Ref="R?"  Part="1"
+AR Path="/54F72FB2/5F88C44B" Ref="R16"  Part="1"
+F 0 "R16" H 2731 2404 50  0000 R CNN
+F 1 "1M 1%" H 2745 2480 50  0000 R CNN
+F 2 "Resistor_SMD:R_0603_1608Metric" H 2790 2450 50  0001 C CNN
+F 3 "~" H 2790 2450 50  0001 C CNN
+F 4 "RT0603BRD071ML" V 2790 2450 50  0001 C CNN "MPN"
+	1    2790 2450
+	0    -1   -1   0
+$EndComp
+Wire Wire Line
+	2585 2315 2625 2315
+Wire Wire Line
+	2875 2315 2930 2315
+Wire Wire Line
+	2690 2450 2625 2450
+Wire Wire Line
+	2625 2450 2625 2315
+Connection ~ 2625 2315
+Wire Wire Line
+	2625 2315 2675 2315
+Wire Wire Line
+	2890 2450 2930 2450
+Wire Wire Line
+	2930 2450 2930 2315
+Connection ~ 2930 2315
+Wire Wire Line
+	2930 2315 2965 2315
+$Comp
+L bottom-board-rescue:C_Small C?
+U 1 1 5F8A2CF0
+P 9440 2650
+AR Path="/54F725AE/5F8A2CF0" Ref="C?"  Part="1"
+AR Path="/54F72FB2/5F8A2CF0" Ref="C93"  Part="1"
+F 0 "C93" V 9490 2700 50  0000 L CNN
+F 1 "1nF" V 9390 2700 50  0000 L CNN
+F 2 "Capacitor_SMD:C_0603_1608Metric" H 9440 2650 60  0001 C CNN
+F 3 "" H 9440 2650 60  0000 C CNN
+F 4 "C0603X7R500-103KNP" H -1460 550 50  0001 C CNN "MPN"
+	1    9440 2650
+	0    1    1    0
+$EndComp
+$Comp
+L bottom-board-rescue:R_Small-Device R?
+U 1 1 5F8A2CF7
+P 9455 2785
+AR Path="/54F72C8D/5F8A2CF7" Ref="R?"  Part="1"
+AR Path="/54F72FB2/5F8A2CF7" Ref="R48"  Part="1"
+F 0 "R48" H 9396 2739 50  0000 R CNN
+F 1 "1M 1%" H 9410 2815 50  0000 R CNN
+F 2 "Resistor_SMD:R_0603_1608Metric" H 9455 2785 50  0001 C CNN
+F 3 "~" H 9455 2785 50  0001 C CNN
+F 4 "RT0603BRD071ML" V 9455 2785 50  0001 C CNN "MPN"
+	1    9455 2785
+	0    -1   -1   0
+$EndComp
+Wire Wire Line
+	9250 2650 9290 2650
+Wire Wire Line
+	9355 2785 9290 2785
+Wire Wire Line
+	9290 2785 9290 2650
+Connection ~ 9290 2650
+Wire Wire Line
+	9290 2650 9340 2650
+Wire Wire Line
+	9540 2650 9605 2650
+Wire Wire Line
+	9605 2785 9605 2650
+Wire Wire Line
+	9555 2785 9605 2785
+Connection ~ 9605 2650
+Wire Wire Line
+	9605 2650 9635 2650
 $EndSCHEMATC

Commit message: change design to 4 layer PCB
Parts:
- P2: MPN 73725-0110BLF -> KUSBX-SLAS1N-B
- R43: MPN RMCF0603JT10K0 -> RMCF0603JT15K0
Changed lines of the file:
@@
 F 2 "Resistor_SMD:R_0603_1608Metric" H 2160 3940 60  0001 C CNN
 F 3 "" H 2160 3940 60  0000 C CNN
-F 4 "RMCF0603JT10K0" H -40 240 50  0001 C CNN "MPN"
+F 4 "RMCF0603JT15K0" H -40 240 50  0001 C CNN "MPN"
 	1    2160 3940
 	1    0    0    -1
@@
 F 2 "Uno:USB_A_Vertical" V 8900 2650 60  0001 C CNN
 F 3 "" V 8900 2650 60  0000 C CNN
-F 4 "73725-0110BLF" H 8950 2750 60  0001 C CNN "MPN"
+F 4 "KUSBX-SLAS1N-B" H 8950 2750 60  0001 C CNN "MPN"
 	1    8950 2750
 	1    0    0    -1

Commit message: minor cleanup
Parts:
- removed U10: RT9742MNGJ5, Package_TO_SOT_SMD:SOT-23-5, symbol bottom-board-rescue:RT9701-Power_Management
- added U10: TPS2001DDBVR, Package_TO_SOT_SMD:SOT-23-5, symbol Power_Management:TPS2041B
Connections:
- net +5V: now also U10.5 (IN)
- net GNDD: now also U10.2 (GND)
- net USB_HOST_DRV: now also U10.4 (~EN)
- net at C52.2, D14.4 (VCC), P2.1 (VCC): now also U10.1 (OUT)
- no-connect marks 0 -> 1
Other:
- moved on the sheet: C51, R46
Changed lines of the file:
@@
-$EndComp
-$Comp
-L bottom-board-rescue:RT9701-Power_Management U10
-U 1 1 55080DFB
-P 7850 3550
-F 0 "U10" H 8050 3800 50  0000 C CNN
-F 1 "RT9742MNGJ5" H 8050 3400 50  0000 C CNN
-F 2 "Package_TO_SOT_SMD:SOT-23-5" H 7850 3550 60  0001 C CNN
-F 3 "https://www.richtek.com/assets/product_file/RT9742/DS9742-07.pdf" H 6950 4600 60  0001 C CNN
-F 4 "RT9742MNGJ5" H 250 0   50  0001 C CNN "MPN"
-	1    7850 3550
-	1    0    0    -1
 $EndComp
 $Comp
 L bottom-board-rescue:R_Small R46
 U 1 1 55083C10
-P 7200 3800
-F 0 "R46" H 7250 3850 50  0000 L CNN
-F 1 "10K" H 7250 3750 50  0000 L CNN
-F 2 "Resistor_SMD:R_0603_1608Metric" H 7200 3800 60  0001 C CNN
-F 3 "~" H 7200 3800 60  0000 C CNN
-F 4 "RR0816P-103-D" H 250 0   50  0001 C CNN "MPN"
-	1    7200 3800
+P 6775 3900
+F 0 "R46" H 6825 3950 50  0000 L CNN
+F 1 "10K" H 6825 3850 50  0000 L CNN
+F 2 "Resistor_SMD:R_0603_1608Metric" H 6775 3900 60  0001 C CNN
+F 3 "~" H 6775 3900 60  0000 C CNN
+F 4 "RR0816P-103-D" H -175 100 50  0001 C CNN "MPN"
+	1    6775 3900
 	1    0    0    -1
 $EndComp
@@
 L bottom-board-rescue:GNDD-power #PWR0180
 U 1 1 55084544
-P 7850 4000
-F 0 "#PWR0180" H 7850 3750 50  0001 C CNN
-F 1 "GNDD" H 7850 3850 50  0000 C CNN
-F 2 "" H 7850 4000 60  0000 C CNN
-F 3 "" H 7850 4000 60  0000 C CNN
-	1    7850 4000
-	1    0    0    -1
-$EndComp
-$Comp
-L bottom-board-rescue:+5V-power #PWR0181
-U 1 1 55085DDA
-P 7250 3000
-F 0 "#PWR0181" H 7250 2850 50  0001 C CNN
-F 1 "+5V" H 7250 3140 50  0000 C CNN
-F 2 "" H 7250 3000 60  0000 C CNN
-F 3 "" H 7250 3000 60  0000 C CNN
-	1    7250 3000
-	1    0    0    -1
-$EndComp
-$Comp
-L bottom-board-rescue:GNDD-power #PWR0182
-U 1 1 5508613A
-P 7750 3150
-F 0 "#PWR0182" H 7750 2900 50  0001 C CNN
-F 1 "GNDD" H 7750 3000 50  0000 C CNN
-F 2 "" H 7750 3150 60  0000 C CNN
-F 3 "" H 7750 3150 60  0000 C CNN
-	1    7750 3150
-	1    0    0    -1
-$EndComp
-$Comp
-L bottom-board-rescue:C_Small C51
-U 1 1 55085190
-P 7500 3100
-F 0 "C51" H 7600 3100 50  0000 L CNN
-F 1 "100nF" H 7550 3000 50  0000 L CNN
-F 2 "Capacitor_SMD:C_0603_1608Metric" H 7500 3100 60  0001 C CNN
-F 3 "" H 7500 3100 60  0000 C CNN
-F 4 "GCM188R71C104KA37D" H 250 0   50  0001 C CNN "MPN"
-	1    7500 3100
-	0    -1   -1   0
+P 7425 4175
+F 0 "#PWR0180" H 7425 3925 50  0001 C CNN
+F 1 "GNDD" H 7425 4025 50  0000 C CNN
+F 2 "" H 7425 4175 60  0000 C CNN
+F 3 "" H 7425 4175 60  0000 C CNN
+	1    7425 4175
+	1    0    0    -1
 $EndComp
 $Comp
@@
 	4750 3700 4750 3800
 Wire Notes Line
-	10800 2150 6250 2150
-Wire Notes Line
 	10800 4450 10800 2150
 Wire Notes Line
-	6250 4450 10800 4450
-Wire Notes Line
-	6250 2150 6250 4450
-Wire Notes Line
 	900  4450 900  2150
 Wire Notes Line
@@
 	900  2150 5550 2150
 Wire Wire Line
-	7750 3100 7750 3150
-Wire Wire Line
-	7600 3100 7750 3100
-Wire Wire Line
-	7400 3100 7250 3100
-Wire Wire Line
-	7250 3000 7250 3100
-Wire Wire Line
-	7250 3450 7350 3450
-Wire Wire Line
-	7200 3700 7200 3550
-Wire Wire Line
-	7200 3950 7850 3950
-Wire Wire Line
-	7200 3900 7200 3950
-Wire Wire Line
-	7850 3750 7850 3950
-Wire Wire Line
-	8500 3550 8500 3450
-Wire Wire Line
-	8350 3550 8500 3550
+	6775 3800 6775 3650
+Wire Wire Line
+	5305 5575 5305 5625
 Wire Wire Line
 	8950 4100 8950 3050
@@
 	4750 3400 4750 3500
 Wire Wire Line
-	8350 3450 8500 3450
-Wire Wire Line
 	10100 3450 10100 3600
 Wire Wire Line
@@
 	9350 3800 9350 4250
 Wire Wire Line
-	7050 3550 7200 3550
+	6625 3650 6775 3650
 Wire Wire Line
 	8750 3050 8750 3450
 Connection ~ 4750 3800
-Connection ~ 7250 3100
-Connection ~ 7200 3550
-Connection ~ 7850 3950
-Connection ~ 8500 3450
+Connection ~ 6775 3650
 Connection ~ 8750 3450
 Connection ~ 1910 3790
@@
 	4750 3800 4750 3850
 Wire Wire Line
-	7250 3100 7250 3450
-Wire Wire Line
-	7200 3550 7350 3550
-Wire Wire Line
-	7850 3950 7850 4000
-Wire Wire Line
-	8500 3450 8750 3450
+	6775 3650 6925 3650
 Wire Wire Line
 	8750 3450 10100 3450
@@
 Wire Wire Line
 	4450 3400 4750 3400
-Text GLabel 7050 3550 0    50   Input ~ 0
+Text GLabel 6625 3650 0    50   Input ~ 0
 USB_HOST_DRV
 $Comp
@@
 Wire Wire Line
 	9605 2650 9635 2650
+$Comp
+L Power_Management:TPS2041B U10
+U 1 1 5FE6A26D
+P 7425 3450
+F 0 "U10" H 7425 3917 50  0000 C CNN
+F 1 "TPS2001DDBVR" H 7425 3826 50  0000 C CNN
+F 2 "Package_TO_SOT_SMD:SOT-23-5" H 7425 3950 50  0001 C CNN
+F 3 "http://www.ti.com/lit/ds/symlink/tps2041.pdf" H 7375 3750 50  0001 C CNN
+F 4 "TPS2001DDBVR" H 7425 3450 50  0001 C CNN "MPN"
+	1    7425 3450
+	1    0    0    -1
+$EndComp
+Wire Notes Line
+	5940 4450 5940 2150
+Wire Notes Line
+	5940 2150 10800 2150
+Wire Notes Line
+	5940 4450 10800 4450
+Wire Wire Line
+	7425 4175 7425 4110
+Wire Wire Line
+	6775 4000 6775 4110
+Wire Wire Line
+	6775 4110 7425 4110
+Connection ~ 7425 4110
+Wire Wire Line
+	7425 4110 7425 4050
+Wire Wire Line
+	7925 3450 8750 3450
+Wire Wire Line
+	7920 3035 7920 3135
+Wire Wire Line
+	8270 3135 8420 3135
+Wire Wire Line
+	8420 3135 8420 3185
+$Comp
+L bottom-board-rescue:C_Small C51
+U 1 1 55085190
+P 8170 3135
+F 0 "C51" H 8270 3135 50  0000 L CNN
+F 1 "100nF" H 8220 3035 50  0000 L CNN
+F 2 "Capacitor_SMD:C_0603_1608Metric" H 8170 3135 60  0001 C CNN
+F 3 "" H 8170 3135 60  0000 C CNN
+F 4 "GCM188R71C104KA37D" H 920 35  50  0001 C CNN "MPN"
+	1    8170 3135
+	0    -1   -1   0
+$EndComp
+$Comp
+L bottom-board-rescue:GNDD-power #PWR0182
+U 1 1 5508613A
+P 8420 3185
+F 0 "#PWR0182" H 8420 2935 50  0001 C CNN
+F 1 "GNDD" H 8420 3035 50  0000 C CNN
+F 2 "" H 8420 3185 60  0000 C CNN
+F 3 "" H 8420 3185 60  0000 C CNN
+	1    8420 3185
+	1    0    0    -1
+$EndComp
+$Comp
+L bottom-board-rescue:+5V-power #PWR0181
+U 1 1 55085DDA
+P 7920 3035
+F 0 "#PWR0181" H 7920 2885 50  0001 C CNN
+F 1 "+5V" H 7920 3175 50  0000 C CNN
+F 2 "" H 7920 3035 60  0000 C CNN
+F 3 "" H 7920 3035 60  0000 C CNN
+	1    7920 3035
+	1    0    0    -1
+$EndComp
+Wire Wire Line
+	7925 3250 7925 3135
+Wire Wire Line
+	7920 3135 7925 3135
+Connection ~ 7925 3135
+Wire Wire Line
+	7925 3135 8070 3135
+NoConn ~ 6925 3250
 $EndSCHEMATC
