File: bottom-board/PCB Source/bottom-board/usb.sch (KiCad schematic (older format))
At the start: 17 parts, among them P1 USB_B, P2 USB_A, U10 TPS2001DDBVR

Commit message: change JFET MPN
Parts:
- U10: MPN AP2822CKETR-G1 -> TPS2001DDBVR
Changed lines of the file:
@@
 F 2 "Package_TO_SOT_SMD:SOT-23-5" H 7425 3950 50  0001 C CNN
 F 3 "http://www.ti.com/lit/ds/symlink/tps2041.pdf" H 7375 3750 50  0001 C CNN
-F 4 "AP2822CKETR-G1" H 7425 3450 50  0001 C CNN "MPN"
+F 4 "TPS2001DDBVR" H 7425 3450 50  0001 C CNN "MPN"
 	1    7425 3450
 	1    0    0    -1

Commit message: change input bias 5->6V, reduce harmonics
Parts:
- U10: MPN TPS2001DDBVR -> AP2822CKETR-G1
Changed lines of the file:
@@
 F 2 "Package_TO_SOT_SMD:SOT-23-5" H 7425 3950 50  0001 C CNN
 F 3 "http://www.ti.com/lit/ds/symlink/tps2041.pdf" H 7375 3750 50  0001 C CNN
-F 4 "TPS2001DDBVR" H 7425 3450 50  0001 C CNN "MPN"
+F 4 "AP2822CKETR-G1" H 7425 3450 50  0001 C CNN "MPN"
 	1    7425 3450
 	1    0    0    -1
