File: bottom-board/PCB Source/bottom-board/_autosave-bottom-board.kicad_pcb (KiCad board)
At the start: 4 copper layers, 194 x 94 mm, 311 parts, among them J1 AS0A823-H4SB-7H, P1 USB_B, P10 JACK_TRS_6PINS, P11 JACK_TRS_6PINS, P12 JACK_TRS_6PINS, P13 RJ45, P14 AudioJack3, P2 USB_A, P3 BARREL_JACK, P5 HMI_DATA, P6 AudioJack3, P7 AudioJack3, P8 SERIAL_DEBUG, P9 JACK_TRS_6PINS, Q1 2N7002, Q10 MMBFJ110, Q12 2N7002, Q13 2N7002, Q2 2N7002, Q3 MMBFJ110, Q4 MMBFJ110, Q5 MMBFJ110, Q6 MMBFJ110, Q7 2N7002, Q8 2N7002, Q9 MMBFJ110, U1 TS2596, U10 TPS2001DDBVR, U11 6N137S, U12 ISL83491, U13 AP2120N-3.3, U2 TL750M10CKVURG3, U3 CS4265, U4 AT24CS08-STUM, U5 LM4562, U6 OPA1678, U7 OPA1678, U8 LM4811, U9 LD1117S50TR_SOT223, X1 24.576MHz

Commit message: update fabrication data
Parts:
- C20, C37, C41, C45, C67, C69, C96: footprint Capacitor_SMD:C_0603_1608Metric -> Capacitor_SMD:C_0805_2012Metric
- moved R3 1.67 mm to (107.1, 119.3)
- moved R69 0.83 mm to (90.2, 117.9)
- moved R87 0.77 mm to (202.7, 113.4)
- moved C4 0.72 mm to (88.6, 117.9)
- moved C17 0.66 mm to (223.5, 90.4)
- moved R95 0.64 mm to (107.0, 72.2)
- moved C45 0.48 mm to (202.6, 111.2)
- moved C20 0.43 mm to (223.2, 92.4)
- moved C47 0.40 mm to (200.0, 110.4)
- moved R107 0.35 mm to (198.4, 111.2)
- moved C67 0.33 mm to (112.3, 76.8)
- moved C36 0.30 mm to (222.6, 80.7)
- moved C69 0.29 mm to (109.0, 69.3)
- moved C96 0.26 mm to (232.5, 93.7)
- moved C37 0.22 mm to (222.6, 82.5)
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Routing:
- net GNDD: track 1385.2 -> 1527.6 mm, vias 146 -> 151
- net CODEC_I2S_SDOUT: track 273.6 -> 238.8 mm
- net +3V3: track 416.6 -> 411.0 mm
- net +10V: track 321.9 -> 317.2 mm
- net IN2_DETECT: track 215.6 -> 211.0 mm
- net Net-(C66-Pad2): track 71.4 -> 67.2 mm
- net +5V: track 219.3 -> 215.3 mm, vias 13 -> 12
- net CODEC_I2S_MCLK: track 9.03 -> 5.03 mm
- net Net-(C65-Pad2): track 68.0 -> 71.2 mm
- net Net-(R3-Pad1): track 125.1 -> 126.8 mm
- net GNDA: track 3507.9 -> 3506.2 mm
- net PM_LEDS_SDA: track 152.8 -> 154.3 mm
- net MIDI_UART_TX: track 177.2 -> 178.5 mm
- net Net-(R95-Pad2): track 8.14 -> 9.14 mm
- net Net-(C47-Pad2): track 4.35 -> 5.32 mm
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Other:
- board text added: "MOD Devices GmbH http://moddevices.com [MDW-ELE-001] MOD Dwarf - Main Board Rev.: MDW-PX30-V1.05 Date: 2021.10.08"
- board text removed: "MOD Devices GmbH http://moddevices.com [MDW-ELE-001] MOD Dwarf - Main Board Rev.: MDW-PX30-V1.05 Date: 2021.XXXX"
