File: bottom-board/PCB Source/bottom-board/audio-codec.sch (KiCad schematic (older format))
At the start: 36 parts, among them U13 AP2120N-3.3, U3 CS4265, X1 24.576MHz

Commit message: update fabrication data
Parts:
- C20, C96: footprint Capacitor_SMD:C_0603_1608Metric -> Capacitor_SMD:C_0805_2012Metric; MPN EMK107BBJ106MA-T -> GRM219R61E106KA12D
Changed lines of the file:
@@
 F 0 "C20" H 7800 4210 50  0000 R CNN
 F 1 "10uF" H 7610 4130 50  0000 L CNN
-F 2 "Capacitor_SMD:C_0603_1608Metric" H 7870 4150 60  0001 C CNN
+F 2 "Capacitor_SMD:C_0805_2012Metric" H 7870 4150 60  0001 C CNN
 F 3 "" H 7870 4150 60  0000 C CNN
-F 4 "EMK107BBJ106MA-T" H 3420 2450 50  0001 C CNN "MPN"
+F 4 "GRM219R61E106KA12D" H 3420 2450 50  0001 C CNN "MPN"
 	1    7870 4150
 	-1   0    0    1
@@
 F 0 "C96" H 5700 4960 50  0000 R CNN
 F 1 "10uF" H 5510 4880 50  0000 L CNN
-F 2 "Capacitor_SMD:C_0603_1608Metric" H 5770 4900 60  0001 C CNN
+F 2 "Capacitor_SMD:C_0805_2012Metric" H 5770 4900 60  0001 C CNN
 F 3 "" H 5770 4900 60  0000 C CNN
-F 4 "EMK107BBJ106MA-T" H 1320 3200 50  0001 C CNN "MPN"
+F 4 "GRM219R61E106KA12D" H 1320 3200 50  0001 C CNN "MPN"
 	1    5770 4900
 	-1   0    0    1
